File: amp_tea2025/amp_tea2025.kicad_pcb (KiCad board)
At the start: 2 copper layers, 18 parts, among them J1 in, J2 SPK, J3 SPK, U1 TEA2025

Commit message: pdf
Parts:
- moved C11 12.7 mm to (45.6, 67.3)
- moved C12 12.7 mm to (86.4, 58.4)
- moved C4 12.7 mm to (80.0, 38.1)
- moved C5 12.7 mm to (43.2, 55.9)
- moved C9 12.7 mm to (62.2, 72.4)
- moved J2 12.7 mm to (30.5, 58.9)
- moved U1 12.7 mm to (61.0, 66.0)
- moved C2 12.7 mm to (41.9, 39.2)
- moved C6 12.7 mm to (28.0, 31.8)
- moved J1 12.7 mm to (76.2, 29.2)
- moved RV1 12.7 mm to (61.0, 29.2)
- moved C1 12.7 mm to (69.8, 50.8)
- moved C10 12.7 mm to (68.7, 68.6)
- moved C13 12.7 mm to (30.5, 50.8)
- moved C3 12.7 mm to (80.1, 48.3)
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
Commit message: all
Parts:
- added J4: power, Connectors_WAGO:WAGO_734_2pin_Straight_RuggedPads, F.Cu at (34.8, 29.2)
- moved C13 7.62 mm to (38.1, 50.8)
- moved C6 7.62 mm to (28.0, 39.4)
Routing:
- net +5V: track 25.9 -> 74.3 mm
- net GND: track 32.9 -> 13.9 mm
- net Net-(C6-Pad1): track 41.8 -> 33.4 mm
- net Net-(C11-Pad1): track 35.0 -> 30.3 mm
- net Net-(J1-Pad3): track 23.6 -> 20.8 mm
Changed lines of the file:
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@@
 (kicad_pcb (version 4) (host pcbnew 4.0.7-e2-6376~61~ubuntu18.04.1)
   (general
-    (links 37)
+    (links 39)
     (no_connects 0)
     (area 23.155 7.934999 102.135715 85.250001)
     (thickness 1.6)
     (drawings 2)
-    (tracks 75)
+    (tracks 73)
     (zones 0)
-    (modules 18)
+    (modules 19)
     (nets 19)
   )
@@
       (subtractmaskfromsilk false)
       (outputformat 4)
-      (mirror true)
+      (mirror false)
       (drillshape 1)
       (scaleselection 1)
@@
   )
   (module Capacitors_THT:CP_Radial_D8.0mm_P5.00mm (layer F.Cu)
-    (at 28.02 31.75)
+    (at 28.02 39.37)
     (descr "CP, Radial series, Radial, pin pitch=5.00mm, , diameter=8mm, Electrolytic Capacitor")
     (tags "CP Radial series Radial pin pitch 5.00mm  diameter 8mm Electrolytic Capacitor")
@@
   )
   (module Capacitors_THT:C_Disc_D9.0mm_W5.0mm_P10.00mm (layer F.Cu)
-    (at 30.48 50.8 90)
+    (at 38.1 50.8 90)
     (descr "C, Disc series, Radial, pin pitch=10.00mm, , diameter*width=9*5.0mm^2, Capacitor, http://www.vishay.com/docs/28535/vy2series.pdf")
     (tags "C Disc series Radial pin pitch 10.00mm  diameter 9mm width 5.0mm Capacitor")
@@
     )
   )
+  (module Connectors_WAGO:WAGO_734_2pin_Straight_RuggedPads (layer F.Cu)
+    (at 34.77006 29.21)
+    (descr "WAGO, Serie 734, Socket, Stiftleiste, 2 polig, 2 pin, rugged Pads, straight, gerade, Date 05Jul2010,")
+    (tags "WAGO, Serie 734, Socket, Stiftleiste, 2 polig, 2 pin, rugged Pads, straight, gerade, Date 05Jul2010,")
+    (fp_text reference J4 (at 0 -6.35) (layer F.SilkS)
+      (effects (font (size 1 1) (thickness 0.15)))
+    )
+    (fp_text value power (at 0 6.35) (layer F.Fab)
+      (effects (font (size 1 1) (thickness 0.15)))
+    )
+    (fp_line (start -4.7498 -2.25044) (end 4.7498 -2.25044) (layer F.SilkS) (width 0.15))
+    (fp_line (start 0.24892 4.24942) (end 0.24892 2.25044) (layer F.SilkS) (width 0.15))
+    (fp_line (start 0.24892 2.25044) (end 1.75006 2.25044) (layer F.SilkS) (width 0.15))
+    (fp_line (start 1.75006 2.25044) (end 1.75006 4.24942) (layer F.SilkS) (width 0.15))
+    (fp_line (start -4.7498 2.25044) (end -1.75006 2.25044) (layer F.SilkS) (width 0.15))
+    (fp_line (start -1.75006 2.25044) (end -1.75006 4.20116) (layer F.SilkS) (width 0.15))
+    (fp_line (start 4.7498 4.24942) (end 4.7498 -4.24942) (layer F.SilkS) (width 0.15))
+    (fp_line (start 4.7498 -4.24942) (end -4.7498 -4.24942) (layer F.SilkS) (width 0.15))
+    (fp_line (start -4.7498 -4.24942) (end -4.7498 4.24942) (layer F.SilkS) (width 0.15))
+    (fp_line (start -4.7498 4.24942) (end 4.7498 4.24942) (layer F.SilkS) (width 0.15))
+    (pad 2 thru_hole oval (at 1.75006 0) (size 1.99898 3.50012) (drill 1.19888) (layers *.Cu *.Mask)
+      (net 13 +5V))
+    (pad 1 thru_hole oval (at -1.75006 0) (size 1.99898 3.50012) (drill 1.19888) (layers *.Cu *.Mask)
+      (net 6 GND))
+  )
   (dimension 62.23 (width 0.3) (layer Dwgs.User)
     (gr_text "2,4500 in" (at 56.515 83.9) (layer Dwgs.User)
@@
   (segment (start 60.96 48.26) (end 80.09 48.26) (width 0.8128) (layer B.Cu) (net 5))
   (segment (start 76.2 29.21) (end 76.2 33.02) (width 0.8128) (layer B.Cu) (net 6))
-  (segment (start 38.1 34.29) (end 38.18 34.21) (width 0.8128) (layer B.Cu) (net 6))
-  (segment (start 38.18 34.21) (end 50.96 34.21) (width 0.8128) (layer B.Cu) (net 6))
-  (segment (start 35.56 31.75) (end 38.1 34.29) (width 0.8128) (layer B.Cu) (net 6))
-  (segment (start 33.02 31.75) (end 35.56 31.75) (width 0.8128) (layer B.Cu) (net 6))
   (segment (start 50.96 29.21) (end 50.96 34.21) (width 0.8128) (layer B.Cu) (net 6))
   (segment (start 53.34 55.88) (end 53.34 58.42) (width 0.8128) (layer B.Cu) (net 6))
@@
   (segment (start 43.18 55.88) (end 43.18 57.4928) (width 0.8128) (layer B.Cu) (net 8))
   (segment (start 43.18 57.4928) (end 46.6472 60.96) (width 0.8128) (layer B.Cu) (net 8))
-  (segment (start 30.48 50.8) (end 33.1 50.8) (width 0.8128) (layer B.Cu) (net 9))
-  (segment (start 33.1 50.8) (end 38.18 55.88) (width 0.8128) (layer B.Cu) (net 9))
+  (segment (start 38.1 50.8) (end 38.1 55.8) (width 0.8128) (layer B.Cu) (net 9))
+  (segment (start 38.1 55.8) (end 38.18 55.88) (width 0.8128) (layer B.Cu) (net 9))
   (segment (start 47.6372 63.5) (end 45.72 65.4172) (width 0.8128) (layer B.Cu) (net 9))
   (segment (start 45.72 65.4172) (end 45.64 65.4972) (width 0.8128) (layer B.Cu) (net 9))
@@
   (segment (start 53.34 63.5) (end 47.6372 63.5) (width 0.8128) (layer B.Cu) (net 9))
   (segment (start 45.64 65.4972) (end 45.64 67.31) (width 0.8128) (layer B.Cu) (net 9))
+  (segment (start 28.02 39.37) (end 28.02 43.26) (width 0.8128) (layer B.Cu) (net 10))
+  (segment (start 31.75 46.99) (end 38.1 46.99) (width 0.8128) (layer B.Cu) (net 10))
+  (segment (start 28.02 43.26) (end 31.75 46.99) (width 0.8128) (layer B.Cu) (net 10))
   (segment (start 38.1 46.99) (end 44.45 53.34) (width 0.8128) (layer B.Cu) (net 10))
   (segment (start 44.45 53.34) (end 53.34 53.34) (width 0.8128) (layer B.Cu) (net 10))
-  (segment (start 30.48 46.99) (end 38.1 46.99) (width 0.8128) (layer B.Cu) (net 10))
-  (segment (start 27.94 44.45) (end 30.48 46.99) (width 0.8128) (layer B.Cu) (net 10))
-  (segment (start 27.94 33.4428) (end 27.94 44.45) (width 0.8128) (layer B.Cu) (net 10))
-  (segment (start 28.02 31.75) (end 28.02 33.3628) (width 0.8128) (layer B.Cu) (net 10))
-  (segment (start 28.02 33.3628) (end 27.94 33.4428) (width 0.8128) (layer B.Cu) (net 10))
   (segment (start 65.1928 60.96) (end 60.96 60.96) (width 0.8128) (layer B.Cu) (net 11))
   (segment (start 67.39 57.15) (end 67.39 58.7628) (width 0.8128) (layer B.Cu) (net 11))
@@
   (segment (start 60.96 63.5) (end 65.3928 63.5) (width 0.8128) (layer B.Cu) (net 12))
   (segment (start 68.66 66.7672) (end 68.66 68.58) (width 0.8128) (layer B.Cu) (net 12))
+  (segment (start 36.52012 29.21) (end 38.33241 29.21) (width 0.8128) (layer B.Cu) (net 13))
+  (segment (start 38.33241 29.21) (end 55.88 46.75759) (width 0.8128) (layer B.Cu) (net 13))
+  (segment (start 55.88 46.75759) (end 55.88 66.04) (width 0.8128) (layer B.Cu) (net 13))
+  (segment (start 55.88 66.04) (end 53.34 66.04) (width 0.8128) (layer B.Cu) (net 13))
   (segment (start 53.34 66.04) (end 53.34 71.28) (width 0.8128) (layer B.Cu) (net 13))
   (segment (start 53.34 71.28) (end 52.23 72.39) (width 0.8128) (layer B.Cu) (net 13))
@@
   (segment (start 66.12 34.21) (end 60.96 34.21) (width 0.8128) (layer B.Cu) (net 16))
   (segment (start 72.69988 29.21) (end 71.12 29.21) (width 0.8128) (layer B.Cu) (net 16))
-  (segment (start 78.74 25.4) (end 79.70012 26.36012) (width 0.8128) (layer B.Cu) (net 17))
-  (segment (start 79.70012 26.36012) (end 79.70012 29.21) (width 0.8128) (layer B.Cu) (net 17))
-  (segment (start 64.77 25.4) (end 78.74 25.4) (width 0.8128) (layer B.Cu) (net 17))
-  (segment (start 60.96 29.21) (end 64.77 25.4) (width 0.8128) (layer B.Cu) (net 17))
+  (segment (start 79.70012 29.21) (end 77.16012 26.67) (width 0.8128) (layer B.Cu) (net 17))
+  (segment (start 77.16012 26.67) (end 63.5 26.67) (width 0.8128) (layer B.Cu) (net 17))
+  (segment (start 63.5 26.67) (end 62.129999 28.040001) (width 0.8128) (layer B.Cu) (net 17))
+  (segment (start 62.129999 28.040001) (end 60.96 29.21) (width 0.8128) (layer B.Cu) (net 17))
   (zone (net 6) (net_name GND) (layer B.Cu) (hatch edge 0.508)
     (connect_pads (clearance 0.508))
