File: amp_tea2025/amp_tea2025.sch (KiCad schematic (older format))
At the start: 18 parts, among them J1 in, J2 SPK, J3 SPK, U1 TEA2025

Commit message: all
Parts:
- added J4: power, Connectors_WAGO:WAGO_734_2pin_Straight_RuggedPads, symbol Conn_01x02
Connections:
- net +5V: now also J4.2 (Pin_2)
- net GND: now also J4.1 (Pin_1)
Changed lines of the file:
@@
 LIBS:valves
 LIBS:MyLibrary
+LIBS:amp_tea2025-cache
 EELAYER 25 0
 EELAYER END
@@
 	6350 2300 6150 2300
 $Comp
-L GND #PWR01
+L GND #PWR4
 U 1 1 5B61741C
 P 6350 2900
-F 0 "#PWR01" H 6350 2650 50  0001 C CNN
+F 0 "#PWR4" H 6350 2650 50  0001 C CNN
 F 1 "GND" H 6350 2750 50  0000 C CNN
 F 2 "" H 6350 2900 50  0001 C CNN
@@
 Connection ~ 7650 2450
 $Comp
-L +5V #PWR02
+L +5V #PWR3
 U 1 1 5B617BC9
 P 6350 1250
-F 0 "#PWR02" H 6350 1100 50  0001 C CNN
+F 0 "#PWR3" H 6350 1100 50  0001 C CNN
 F 1 "+5V" H 6350 1390 50  0000 C CNN
 F 2 "" H 6350 1250 50  0001 C CNN
@@
 $EndComp
 Wire Wire Line
-	6500 1300 6350 1300
+	5650 1300 6500 1300
 Connection ~ 6350 1300
 $Comp
-L GND #PWR03
+L GND #PWR5
 U 1 1 5B617CF5
 P 7150 1300
-F 0 "#PWR03" H 7150 1050 50  0001 C CNN
+F 0 "#PWR5" H 7150 1050 50  0001 C CNN
 F 1 "GND" H 7150 1150 50  0000 C CNN
 F 2 "" H 7150 1300 50  0001 C CNN
@@
 $EndComp
 $Comp
-L GND #PWR04
+L GND #PWR1
 U 1 1 5B618C90
 P 3750 2350
-F 0 "#PWR04" H 3750 2100 50  0001 C CNN
+F 0 "#PWR1" H 3750 2100 50  0001 C CNN
 F 1 "GND" H 3750 2200 50  0000 C CNN
 F 2 "" H 3750 2350 50  0001 C CNN
@@
 Wire Wire Line
 	3600 1400 3600 1750
+$Comp
+L Conn_01x02 J4
+U 1 1 5B643377
+P 5550 800
+F 0 "J4" H 5550 900 50  0000 C CNN
+F 1 "power" H 5550 600 50  0000 C CNN
+F 2 "Connectors_WAGO:WAGO_734_2pin_Straight_RuggedPads" H 5550 800 50  0001 C CNN
+F 3 "" H 5550 800 50  0001 C CNN
+	1    5550 800
+	0    -1   -1   0
+$EndComp
+Wire Wire Line
+	5650 1000 5650 1300
+$Comp
+L GND #PWR2
+U 1 1 5B6434A2
+P 5550 1100
+F 0 "#PWR2" H 5550 850 50  0001 C CNN
+F 1 "GND" H 5550 950 50  0000 C CNN
+F 2 "" H 5550 1100 50  0001 C CNN
+F 3 "" H 5550 1100 50  0001 C CNN
+	1    5550 1100
+	1    0    0    -1
+$EndComp
+Wire Wire Line
+	5550 1000 5550 1100
 $EndSCHEMATC
