File: i2c_portexpander/_saved_i2c_portexpander.sch (KiCad schematic (older format))
At the start: 19 parts, among them J1 i2c, J2 ttl_out, J3 RSW1, J4 RSW2, J5 RSW3, J6 RSW4, J7 power, P1 RELAY, P2 RELAY, P3 RELAY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

Commit message: i2c
Parts:
- added R4, R5: 4k7, Resistors_SMD:R_0805_HandSoldering, symbol R
Connections:
- net +VSW: now also R4.1, R5.1
- net at J1.1 (Pin_1), U1.14 (SCL): now also R4.2
- net at J1.2 (Pin_2), U1.15 (SDA): now also R5.2
Changed lines of the file:
@@
 	4850 3800 7900 3800
 Connection ~ 7900 3600
+$Comp
+L R R4
+U 1 1 5B6975AF
+P 2200 900
+F 0 "R4" V 2280 900 50  0000 C CNN
+F 1 "4k7" V 2200 900 50  0000 C CNN
+F 2 "Resistors_SMD:R_0805_HandSoldering" V 2130 900 50  0001 C CNN
+F 3 "" H 2200 900 50  0001 C CNN
+	1    2200 900
+	1    0    0    -1
+$EndComp
+$Comp
+L R R5
+U 1 1 5B69785D
+P 2400 900
+F 0 "R5" V 2480 900 50  0000 C CNN
+F 1 "4k7" V 2400 900 50  0000 C CNN
+F 2 "Resistors_SMD:R_0805_HandSoldering" V 2330 900 50  0001 C CNN
+F 3 "" H 2400 900 50  0001 C CNN
+	1    2400 900
+	1    0    0    -1
+$EndComp
+Wire Wire Line
+	2200 750  2200 700
+Connection ~ 2200 700
+Wire Wire Line
+	2400 750  2400 700
+Connection ~ 2400 700
+Wire Wire Line
+	2200 1050 2200 1100
+Connection ~ 2200 1100
+Wire Wire Line
+	2400 1050 2400 1350
+Connection ~ 2400 1350
 $EndSCHEMATC
