File: i2c_portexpander/i2c_portexpander.kicad_pcb (KiCad board)
At the start: 2 copper layers, 16 parts, among them J1 Conn_01x02_Male, J2 Screw_Terminal_01x04, J3 Screw_Terminal_01x02, J4 Screw_Terminal_01x02, J5 Screw_Terminal_01x02, J6 Screw_Terminal_01x02, P1 RELAY831-1A, P2 RELAY831-1A, P3 RELAY831-1A, P4 RELAY831-1A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

Commit message: all
Parts:
- moved J2 70.8 mm to (128.1, 44.5)
- moved R1 28.4 mm to (114.4, 73.7), turned to 180 degrees
- moved J1 24.4 mm to (132.1, 99.1)
- moved SW1 22.5 mm to (113.0, 81.3)
- moved R3 20.7 mm to (115.7, 88.9), turned to 180 degrees
- moved R2 14.2 mm to (113.1, 92.7)
- moved J5 2.80 mm to (179.1, 47.0), turned to 90 degrees
- moved J3 2.80 mm to (179.1, 79.9), turned to 90 degrees
- moved J4 2.73 mm to (179.1, 63.4), turned to 90 degrees
- moved J6 2.73 mm to (179.1, 96.4), turned to 90 degrees
- moved U2 1.01 mm to (127.3, 64.8)
Routing:
- net Net-(R2-Pad1): track 0.00 -> 19.9 mm
- net Net-(R1-Pad1): track 0.00 -> 12.5 mm
- net Net-(R3-Pad1): track 0.00 -> 10.6 mm
- net Net-(U1-Pad11): track 14.9 -> 21.3 mm
- net Net-(U1-Pad4): track 12.4 -> 18.4 mm
- net Net-(U1-Pad9): track 19.0 -> 24.4 mm
- net Net-(U1-Pad10): track 18.2 -> 22.5 mm
- net Net-(U1-Pad7): track 19.0 -> 23.4 mm
- net Net-(U1-Pad6): track 17.2 -> 21.6 mm
- net Net-(U1-Pad5): track 15.5 -> 19.8 mm
- net +VSW: track 0.00 -> 3.88 mm
- net Net-(P2-Pad1): track 0.00 -> 0.99 mm
Other:
- rule trace_min: 0.2 -> 0.1524

Commit message: i2c
Parts:
- added C1: 0.1, Capacitors_SMD:C_1206_HandSoldering, F.Cu at (36.8, 61.0)
- added C2: 0.1, Capacitors_SMD:C_1206_HandSoldering, F.Cu at (35.6, 47.0)
- added J7: power, Connectors_Molex:Molex_KK-6410-02_02x2.54mm_Straight, F.Cu at (24.1, 80.0)
- added R4: 4k7, Resistors_SMD:R_0805_HandSoldering, F.Cu at (34.3, 72.3)
- added R5: 4k7, Resistors_SMD:R_0805_HandSoldering, F.Cu at (38.1, 72.5)
- J1: value Conn_01x02_Male -> i2c
- J2: value Screw_Terminal_01x04 -> ttl_out
- J3: value Screw_Terminal_01x02 -> RSW1
- J4: value Screw_Terminal_01x02 -> RSW2
- J5: value Screw_Terminal_01x02 -> RSW3
- J6: value Screw_Terminal_01x02 -> RSW4
- P1, P2, P3, P4: value RELAY831-1A -> RELAY
- SW1: value SW_DIP_x03 -> i2c_addr
- moved J6 133.5 mm to (68.6, 21.5), turned to 270 degrees
- moved P4 129.8 mm to (49.5, 26.8)
- moved J5 111.0 mm to (68.3, 38.9), turned to 270 degrees
- moved J4 110.7 mm to (68.6, 56.2), turned to 270 degrees
- moved J3 110.7 mm to (68.6, 73.6), turned to 270 degrees
- moved P3 108.7 mm to (49.5, 44.2)
- moved P2 108.6 mm to (49.5, 61.5)
- moved P1 108.6 mm to (49.5, 78.9)
- moved U1 104.2 mm to (28.4, 52.7)
- moved U2 103.2 mm to (27.9, 36.8)
- moved R2 101.3 mm to (20.3, 52.1), turned to 270 degrees
- moved J1 99.6 mm to (34.3, 80.0)
- moved J2 98.6 mm to (31.9, 22.9)
- moved R1 97.8 mm to (20.3, 46.9), turned to 90 degrees
- moved R3 90.1 mm to (30.4, 59.7), turned to 0 degrees
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Connections:
- net Net-(SW1-Pad1) renamed GND
- J2 pad 1: Net-(J2-Pad1) -> +VSW
- P4 pad 1: Net-(J2-Pad1) -> Net-(P4-Pad1)
- U2 pad 13: Net-(J2-Pad1) -> Net-(P4-Pad1)
Routing:
- net +VSW: track 3.88 -> 243.8 mm, vias 0 -> 4
- net Net-(P1-Pad1): track 0.00 -> 62.7 mm
- net GND: track 0.00 -> 53.9 mm, vias 0 -> 1
- net Net-(P2-Pad1): track 0.99 -> 46.2 mm
- net Net-(J1-Pad2): track 0.00 -> 34.4 mm
- net Net-(J1-Pad1): track 0.00 -> 31.6 mm
- net Net-(P3-Pad1): track 0.45 -> 29.3 mm
- net Net-(J5-Pad2): track 0.00 -> 26.3 mm
- net Net-(J6-Pad2): track 0.00 -> 25.4 mm
- net Net-(J4-Pad2): track 0.00 -> 25.4 mm
- net Net-(J3-Pad2): track 0.00 -> 25.4 mm
- net Net-(P4-Pad1): track 0.00 -> 20.5 mm
- net Net-(J2-Pad4): track 0.00 -> 12.9 mm
- net Net-(J2-Pad2): track 0.00 -> 12.7 mm
- net Net-(J2-Pad3): track 0.00 -> 12.0 mm
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- added copper zone on B.Cu, net GND
- added copper zone on F.Cu, net GND
