File: i2c_portexpander/i2c_portexpander.sch (KiCad schematic (older format))
At the start: 16 parts, among them J1 Conn_01x02_Male, J2 Screw_Terminal_01x04, J3 Screw_Terminal_01x02, J4 Screw_Terminal_01x02, J5 Screw_Terminal_01x02, J6 Screw_Terminal_01x02, P1 RELAY831-1A, P2 RELAY831-1A, P3 RELAY831-1A, P4 RELAY831-1A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

Commit message: i2c
Parts:
- added C1, C2: 0.1, Capacitors_SMD:C_1206_HandSoldering, symbol C_Small
- added J7: power, Connectors_Molex:Molex_KK-6410-02_02x2.54mm_Straight, symbol Conn_01x02_Male
- added R? (x2): 4k7, Resistors_SMD:R_0805_HandSoldering, symbol R
- J1: value Conn_01x02_Male -> i2c
- J2: value Screw_Terminal_01x04 -> ttl_out
- J3: value Screw_Terminal_01x02 -> RSW1
- J4: value Screw_Terminal_01x02 -> RSW2
- J5: value Screw_Terminal_01x02 -> RSW3
- J6: value Screw_Terminal_01x02 -> RSW4
- P1, P2, P3, P4: value RELAY831-1A -> RELAY
- SW1: value SW_DIP_x03 -> i2c_addr
Connections:
- net +VSW: now also J2.1 (Pin_1), C1.2, C2.1, J7.1 (Pin_1), R?.1, R?.1
- net at J1.1 (Pin_1), U1.14 (SCL): now also R?.2
- net at J1.2 (Pin_2), U1.15 (SDA): now also R?.2
- net GND: now reaches SW1.1, SW1.2, SW1.3, U1.8 (VSS), U2.8 (GND)
- net GND: now also C1.1, C2.2, J7.2 (Pin_2)
- net at P4.1, U2.13 (O4): no longer J2.1 (Pin_1)
Changed lines of the file:
@@
 P 6100 1100
 F 0 "P1" H 6300 800 60  0000 C CNN
-F 1 "RELAY831-1A" H 6750 1250 60  0000 C CNN
+F 1 "RELAY" H 6750 1250 60  0000 C CNN
 F 2 "mih-library:Relay-841-1A" H 6750 1250 60  0001 C CNN
 F 3 "" H 6750 1250 60  0001 C CNN
@@
 P 6100 1850
 F 0 "P2" H 6300 1550 60  0000 C CNN
-F 1 "RELAY831-1A" H 6750 2000 60  0000 C CNN
+F 1 "RELAY" H 6750 2000 60  0000 C CNN
 F 2 "mih-library:Relay-841-1A" H 6750 2000 60  0001 C CNN
 F 3 "" H 6750 2000 60  0001 C CNN
@@
 P 6100 2650
 F 0 "P3" H 6300 2350 60  0000 C CNN
-F 1 "RELAY831-1A" H 6750 2800 60  0000 C CNN
+F 1 "RELAY" H 6750 2800 60  0000 C CNN
 F 2 "mih-library:Relay-841-1A" H 6750 2800 60  0001 C CNN
 F 3 "" H 6750 2800 60  0001 C CNN
@@
 P 6100 3400
 F 0 "P4" H 6300 3100 60  0000 C CNN
-F 1 "RELAY831-1A" H 6750 3550 60  0000 C CNN
+F 1 "RELAY" H 6750 3550 60  0000 C CNN
 F 2 "mih-library:Relay-841-1A" H 6750 3550 60  0001 C CNN
 F 3 "" H 6750 3550 60  0001 C CNN
@@
 P 7000 900
 F 0 "J3" H 7000 1000 50  0000 C CNN
-F 1 "Screw_Terminal_01x02" H 7000 700 50  0000 C CNN
+F 1 "RSW1" H 7000 700 50  0000 C CNN
 F 2 "Connectors_Terminal_Blocks:TerminalBlock_Pheonix_MKDS1.5-2pol" H 7000 900 50  0001 C CNN
 F 3 "" H 7000 900 50  0001 C CNN
@@
 P 7050 1650
 F 0 "J4" H 7050 1750 50  0000 C CNN
-F 1 "Screw_Terminal_01x02" H 7050 1450 50  0000 C CNN
+F 1 "RSW2" H 7050 1450 50  0000 C CNN
 F 2 "Connectors_Terminal_Blocks:TerminalBlock_Pheonix_MKDS1.5-2pol" H 7050 1650 50  0001 C CNN
 F 3 "" H 7050 1650 50  0001 C CNN
@@
 P 7050 2450
 F 0 "J5" H 7050 2550 50  0000 C CNN
-F 1 "Screw_Terminal_01x02" H 7050 2250 50  0000 C CNN
+F 1 "RSW3" H 7050 2250 50  0000 C CNN
 F 2 "Connectors_Terminal_Blocks:TerminalBlock_Pheonix_MKDS1.5-2pol" H 7050 2450 50  0001 C CNN
 F 3 "" H 7050 2450 50  0001 C CNN
@@
 P 7050 3200
 F 0 "J6" H 7050 3300 50  0000 C CNN
-F 1 "Screw_Terminal_01x02" H 7050 3000 50  0000 C CNN
+F 1 "RSW4" H 7050 3000 50  0000 C CNN
 F 2 "Connectors_Terminal_Blocks:TerminalBlock_Pheonix_MKDS1.5-2pol" H 7050 3200 50  0001 C CNN
 F 3 "" H 7050 3200 50  0001 C CNN
@@
 P 1750 1750
 F 0 "SW1" H 1750 2100 50  0000 C CNN
-F 1 "SW_DIP_x03" H 1750 1600 50  0000 C CNN
+F 1 "i2c_addr" H 1750 1600 50  0000 C CNN
 F 2 "Buttons_Switches_SMD:SW_DIP_x3_W8.61mm_Slide_LowProfile" H 1750 1750 50  0001 C CNN
 F 3 "" H 1750 1750 50  0001 C CNN
@@
 	2050 1550 2550 1550
 Wire Wire Line
-	2550 1650 2050 1650
+	2050 1650 2550 1650
 Wire Wire Line
 	2050 1750 2550 1750
@@
 Connection ~ 1450 1650
 Wire Wire Line
-	3050 2350 3050 2550
+	3050 2350 3050 2850
 Wire Wire Line
 	1450 2550 4650 2550
@@
 Connection ~ 2250 2150
 $Comp
-L +VSW #PWR2
+L +VSW #PWR3
 U 1 1 5B4DF5CF
 P 3050 850
-F 0 "#PWR2" H 3050 700 50  0001 C CNN
+F 0 "#PWR3" H 3050 700 50  0001 C CNN
 F 1 "+VSW" H 3050 990 50  0000 C CNN
 F 2 "" H 3050 850 50  0001 C CNN
@@
 P 1600 1100
 F 0 "J1" H 1600 1200 50  0000 C CNN
-F 1 "Conn_01x02_Male" H 1600 900 50  0000 C CNN
+F 1 "i2c" H 1600 900 50  0000 C CNN
 F 2 "Connectors_Molex:Molex_KK-6410-02_02x2.54mm_Straight" H 1600 1100 50  0001 C CNN
 F 3 "" H 1600 1100 50  0001 C CNN
@@
 Connection ~ 3050 2550
 $Comp
-L +VSW #PWR3
+L +VSW #PWR7
 U 1 1 5B4DFDFC
 P 7900 1250
-F 0 "#PWR3" H 7900 1100 50  0001 C CNN
+F 0 "#PWR7" H 7900 1100 50  0001 C CNN
 F 1 "+VSW" H 7900 1390 50  0000 C CNN
 F 2 "" H 7900 1250 50  0001 C CNN
@@
 $EndComp
 Wire Wire Line
-	7900 1250 7900 3600
+	7900 1250 7900 3800
 Wire Wire Line
 	6500 1300 7600 1300
@@
 P 4650 3100
 F 0 "J2" H 4650 3300 50  0000 C CNN
-F 1 "Screw_Terminal_01x04" H 4650 2800 50  0000 C CNN
+F 1 "ttl_out" H 4650 2800 50  0000 C CNN
 F 2 "Connectors_WAGO:WAGO_734_4pin_Straight" H 4650 3100 50  0001 C CNN
 F 3 "" H 4650 3100 50  0001 C CNN
@@
 Wire Wire Line
 	5200 3100 4850 3100
-Wire Wire Line
-	4850 3200 5450 3200
 Connection ~ 5450 3200
+$Comp
+L C_Small C2
+U 1 1 5B6959A1
+P 4300 2400
+F 0 "C2" H 4310 2470 50  0000 L CNN
+F 1 "0.1" H 4310 2320 50  0000 L CNN
+F 2 "Capacitors_SMD:C_1206_HandSoldering" H 4300 2400 50  0001 C CNN
+F 3 "" H 4300 2400 50  0001 C CNN
+	1    4300 2400
+	0    -1   -1   0
+$EndComp
+$Comp
+L C_Small C1
+U 1 1 5B695A40
+P 3300 850
+F 0 "C1" H 3310 920 50  0000 L CNN
+F 1 "0.1" H 3310 770 50  0000 L CNN
+F 2 "Capacitors_SMD:C_1206_HandSoldering" H 3300 850 50  0001 C CNN
+F 3 "" H 3300 850 50  0001 C CNN
+	1    3300 850
+	0    1    1    0
+$EndComp
+Wire Wire Line
+	2800 850  3200 850
+$Comp
+L GND #PWR4
+U 1 1 5B695B93
+P 3050 2850
+F 0 "#PWR4" H 3050 2600 50  0001 C CNN
+F 1 "GND" H 3050 2700 50  0000 C CNN
+F 2 "" H 3050 2850 50  0001 C CNN
+F 3 "" H 3050 2850 50  0001 C CNN
+	1    3050 2850
+	1    0    0    -1
+$EndComp
+$Comp
+L GND #PWR5
+U 1 1 5B695BDB
+P 3650 850
+F 0 "#PWR5" H 3650 600 50  0001 C CNN
+F 1 "GND" H 3650 700 50  0000 C CNN
+F 2 "" H 3650 850 50  0001 C CNN
+F 3 "" H 3650 850 50  0001 C CNN
+	1    3650 850
+	1    0    0    -1
+$EndComp
+$Comp
+L +VSW #PWR6
+U 1 1 5B695C1C
+P 4100 2300
+F 0 "#PWR6" H 4100 2150 50  0001 C CNN
+F 1 "+VSW" H 4100 2440 50  0000 C CNN
+F 2 "" H 4100 2300 50  0001 C CNN
+F 3 "" H 4100 2300 50  0001 C CNN
+	1    4100 2300
+	1    0    0    -1
+$EndComp
+Wire Wire Line
+	4400 2400 4650 2400
+Connection ~ 4650 2400
+Wire Wire Line
+	4100 2300 4200 2300
+Wire Wire Line
+	4200 2300 4200 2400
+Wire Wire Line
+	3400 850  3650 850
+Connection ~ 3450 850
+Connection ~ 3050 850
+$Comp
+L Conn_01x02_Male J7
+U 1 1 5B6965B2
+P 1600 700
+F 0 "J7" H 1600 800 50  0000 C CNN
+F 1 "power" H 1600 500 50  0000 C CNN
+F 2 "Connectors_Molex:Molex_KK-6410-02_02x2.54mm_Straight" H 1600 700 50  0001 C CNN
+F 3 "" H 1600 700 50  0001 C CNN
+	1    1600 700
+	1    0    0    -1
+$EndComp
+Wire Wire Line
+	1800 700  2800 700
+Wire Wire Line
+	2800 700  2800 850
+$Comp
+L GND #PWR2
+U 1 1 5B696AAE
+P 2050 800
+F 0 "#PWR2" H 2050 550 50  0001 C CNN
+F 1 "GND" H 2050 650 50  0000 C CNN
+F 2 "" H 2050 800 50  0001 C CNN
+F 3 "" H 2050 800 50  0001 C CNN
+	1    2050 800
+	1    0    0    -1
+$EndComp
+Wire Wire Line
+	1800 800  2050 800
+Wire Wire Line
+	4850 3200 4850 3800
+Wire Wire Line
+	4850 3800 7900 3800
+Connection ~ 7900 3600
+$Comp
+L R R?
+U 1 1 5B6975AF
+P 2200 900
+F 0 "R?" V 2280 900 50  0000 C CNN
+F 1 "4k7" V 2200 900 50  0000 C CNN
+F 2 "Resistors_SMD:R_0805_HandSoldering" V 2130 900 50  0001 C CNN
+F 3 "" H 2200 900 50  0001 C CNN
+	1    2200 900
+	1    0    0    -1
+$EndComp
+$Comp
+L R R?
+U 1 1 5B69785D
+P 2400 900
+F 0 "R?" V 2480 900 50  0000 C CNN
+F 1 "4k7" V 2400 900 50  0000 C CNN
+F 2 "Resistors_SMD:R_0805_HandSoldering" V 2330 900 50  0001 C CNN
+F 3 "" H 2400 900 50  0001 C CNN
+	1    2400 900
+	1    0    0    -1
+$EndComp
+Wire Wire Line
+	2200 750  2200 700
+Connection ~ 2200 700
+Wire Wire Line
+	2400 750  2400 700
+Connection ~ 2400 700
+Wire Wire Line
+	2200 1050 2200 1100
+Connection ~ 2200 1100
+Wire Wire Line
+	2400 1050 2400 1350
+Connection ~ 2400 1350
 $EndSCHEMATC
