File: Усилитель1557q/Усилитель1557q.kicad_pcb (KiCad board)
At the start: 2 copper layers, 50 x 50 mm, 9 parts, among them J1 INPUT, J2 Power, J3 OUT1, J4 OUT2, U1 TDA1557Q

Commit message: 1557q-improved
Parts:
- added C4: 4200mF, Capacitors_THT:CP_Radial_D13.0mm_P5.00mm, F.Cu at (61.0, 78.7)
- added R1: 220k, Resistors_THT:R_Axial_DIN0204_L3.6mm_D1.6mm_P7.62mm_Horizontal, F.Cu at (71.1, 98.0)
- added R2: 220k, Resistors_THT:R_Axial_DIN0204_L3.6mm_D1.6mm_P7.62mm_Horizontal, F.Cu at (71.1, 93.0)
- moved C3 6.48 mm to (72.4, 78.7)
- moved J3 6.35 mm to (85.2, 74.9)
- moved J2 6.35 mm to (49.5, 78.7)
Connections:
- RV1 pad 2: Net-(C1-Pad2) -> Net-(R2-Pad2)
- RV1 pad 5: Net-(C2-Pad2) -> Net-(R1-Pad2)
Routing:
- net GNDPWR: track 44.9 -> 0.00 mm
- net Net-(C1-Pad2): track 22.2 -> 5.38 mm
- net +12VA: track 94.6 -> 107.3 mm
- net Net-(R2-Pad2): track 0.00 -> 12.5 mm
- net Net-(C2-Pad2): track 17.2 -> 4.88 mm
- net Net-(R1-Pad2): track 0.00 -> 8.70 mm
- net Net-(J3-Pad1): track 25.9 -> 21.0 mm
- net Net-(J1-Pad1): track 34.6 -> 39.2 mm
- net Net-(J1-Pad2): track 72.8 -> 76.3 mm
- net Net-(J3-Pad2): track 25.9 -> 23.2 mm
- added copper zone on B.Cu, net GNDPWR
