File: Усилитель1557q/Усилитель1557q.sch (KiCad schematic (older format))
At the start: 10 parts, among them J1 INPUT, J2 Power, J3 OUT1, J4 OUT2, U1 TDA1557Q

Commit message: 1557q-improved
Parts:
- added R1, R2: 220k, Resistors_THT:R_Axial_DIN0204_L3.6mm_D1.6mm_P7.62mm_Horizontal, symbol R_Small
Connections:
- net at C1.2: now also R2.1; no longer RV1.2
- net at RV1.5: now also R1.2; no longer C2.2
- new net: R2.2, RV1.2
- new net: C2.2, R1.1
Changed lines of the file:
@@
 $EndComp
 $Comp
-L GNDPWR #PWR2
+L GNDPWR #PWR01
 U 1 1 5B5ED18A
 P 5650 3750
-F 0 "#PWR2" H 5650 3550 50  0001 C CNN
+F 0 "#PWR01" H 5650 3550 50  0001 C CNN
 F 1 "GNDPWR" H 5650 3620 50  0000 C CNN
 F 2 "" H 5650 3700 50  0001 C CNN
@@
 $EndComp
 $Comp
-L +12VA #PWR3
+L +12VA #PWR02
 U 1 1 5B5ED31F
 P 6250 1050
-F 0 "#PWR3" H 6250 900 50  0001 C CNN
+F 0 "#PWR02" H 6250 900 50  0001 C CNN
 F 1 "+12VA" H 6250 1190 50  0000 C CNN
 F 2 "" H 6250 1050 50  0001 C CNN
@@
 $EndComp
 $Comp
-L +12VA #PWR4
+L +12VA #PWR03
 U 1 1 5B5EDCB5
 P 6850 1050
-F 0 "#PWR4" H 6850 900 50  0001 C CNN
+F 0 "#PWR03" H 6850 900 50  0001 C CNN
 F 1 "+12VA" H 6850 1190 50  0000 C CNN
 F 2 "" H 6850 1050 50  0001 C CNN
@@
 $EndComp
 $Comp
-L GNDPWR #PWR1
+L GNDPWR #PWR04
 U 1 1 5B5EDCE0
 P 5150 1100
-F 0 "#PWR1" H 5150 900 50  0001 C CNN
+F 0 "#PWR04" H 5150 900 50  0001 C CNN
 F 1 "GNDPWR" H 5150 970 50  0000 C CNN
 F 2 "" H 5150 1050 50  0001 C CNN
@@
 $EndComp
 Wire Wire Line
-	5500 1050 5150 1050
+	5150 1050 5500 1050
 Wire Wire Line
 	5150 650  5150 1100
 Wire Wire Line
-	6850 1050 6500 1050
-Wire Wire Line
-	6500 1050 6500 750
+	6500 1050 6850 1050
+Wire Wire Line
+	6500 750  6500 1050
 Wire Wire Line
 	6500 650  5150 650
@@
 Connection ~ 3450 2050
 Wire Wire Line
-	3900 2350 4250 2350
-Wire Wire Line
 	4250 2350 4250 2200
 Wire Wire Line
 	4250 2200 4450 2200
-Wire Wire Line
-	3900 1850 4450 1850
 Wire Wire Line
 	4450 1850 4450 1950
@@
 	5700 800  6500 800
 Connection ~ 6500 800
+$Comp
+L R_Small R2
+U 1 1 5B74120C
+P 4150 1850
+F 0 "R2" H 4180 1870 50  0000 L CNN
+F 1 "220k" H 4180 1810 50  0000 L CNN
+F 2 "Resistors_THT:R_Axial_DIN0204_L3.6mm_D1.6mm_P7.62mm_Horizontal" H 4150 1850 50  0001 C CNN
+F 3 "" H 4150 1850 50  0001 C CNN
+	1    4150 1850
+	0    1    1    0
+$EndComp
+Wire Wire Line
+	4250 1850 4450 1850
+Wire Wire Line
+	4050 1850 3900 1850
+$Comp
+L R_Small R1
+U 1 1 5B741358
+P 4050 2350
+F 0 "R1" H 4080 2370 50  0000 L CNN
+F 1 "220k" H 4080 2310 50  0000 L CNN
+F 2 "Resistors_THT:R_Axial_DIN0204_L3.6mm_D1.6mm_P7.62mm_Horizontal" H 4050 2350 50  0001 C CNN
+F 3 "" H 4050 2350 50  0001 C CNN
+	1    4050 2350
+	0    1    1    0
+$EndComp
+Wire Wire Line
+	3900 2350 3950 2350
+Wire Wire Line
+	4150 2350 4250 2350
 $EndSCHEMATC
