File: waterlock/controller.sch (KiCad schematic (older format))
At the start: 29 parts, among them CON1 AVR-ISP-10, CON2 AVR-ISP-6, J1 v5, J2 v12, J3 m1, J4 m2, J5 Battery, J6 L1, J7 L2, SW1 Turn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

Commit message: firmware start
Parts:
- removed C1, C2: 10mF, Capacitors_THT:CP_Radial_D5.0mm_P2.50mm, symbol CP_Small
- removed CON2: AVR-ISP-6, Connectors:IDC_Header_Straight_6pins, symbol AVR-ISP-6
- SW1: footprint Buttons_Switches_SMD:SW_SPST_PTS645 -> Buttons_Switches_THT:SW_PUSH_6mm_h8.5mm
Connections:
- wire segments 116 -> 106
Changed lines of the file:
@@
 	7300 2150 7300 2200
 $Comp
-L GND #PWR9
+L GND #PWR01
 U 1 1 5B7A7AAC
 P 6600 3050
-F 0 "#PWR9" H 6600 2800 50  0001 C CNN
+F 0 "#PWR01" H 6600 2800 50  0001 C CNN
 F 1 "GND" H 6600 2900 50  0000 C CNN
 F 2 "" H 6600 3050 50  0001 C CNN
@@
 Connection ~ 6650 2800
 $Comp
-L +12V #PWR10
+L +12V #PWR02
 U 1 1 5B7A7C3C
 P 7850 700
-F 0 "#PWR10" H 7850 550 50  0001 C CNN
+F 0 "#PWR02" H 7850 550 50  0001 C CNN
 F 1 "+12V" H 7850 840 50  0000 C CNN
 F 2 "" H 7850 700 50  0001 C CNN
@@
 $EndComp
 $Comp
-L +5V #PWR5
+L +5V #PWR03
 U 1 1 5B7A7CE0
 P 4550 650
-F 0 "#PWR5" H 4550 500 50  0001 C CNN
+F 0 "#PWR03" H 4550 500 50  0001 C CNN
 F 1 "+5V" H 4550 790 50  0000 C CNN
 F 2 "" H 4550 650 50  0001 C CNN
@@
 	1650 650  5200 650
 $Comp
-L GND #PWR6
+L GND #PWR04
 U 1 1 5B7A7EE1
 P 4850 750
-F 0 "#PWR6" H 4850 500 50  0001 C CNN
+F 0 "#PWR04" H 4850 500 50  0001 C CNN
 F 1 "GND" H 4850 600 50  0000 C CNN
 F 2 "" H 4850 750 50  0001 C CNN
@@
 $EndComp
 $Comp
-L GND #PWR12
+L GND #PWR05
 U 1 1 5B7A7EFE
 P 8150 800
-F 0 "#PWR12" H 8150 550 50  0001 C CNN
+F 0 "#PWR05" H 8150 550 50  0001 C CNN
 F 1 "GND" H 8150 650 50  0000 C CNN
 F 2 "" H 8150 800 50  0001 C CNN
@@
 $EndComp
 $Comp
-L +12V #PWR11
+L +12V #PWR06
 U 1 1 5B7C12D6
 P 8050 4750
-F 0 "#PWR11" H 8050 4600 50  0001 C CNN
+F 0 "#PWR06" H 8050 4600 50  0001 C CNN
 F 1 "+12V" H 8050 4890 50  0000 C CNN
 F 2 "" H 8050 4750 50  0001 C CNN
@@
 	8600 4950 8850 4950
 $Comp
-L GND #PWR13
+L GND #PWR07
 U 1 1 5B7C1985
 P 8600 5050
-F 0 "#PWR13" H 8600 4800 50  0001 C CNN
+F 0 "#PWR07" H 8600 4800 50  0001 C CNN
 F 1 "GND" H 8600 4900 50  0000 C CNN
 F 2 "" H 8600 5050 50  0001 C CNN
@@
 Connection ~ 4550 650
 $Comp
-L GND #PWR4
+L GND #PWR08
 U 1 1 5B7E4EA7
 P 3150 4300
-F 0 "#PWR4" H 3150 4050 50  0001 C CNN
+F 0 "#PWR08" H 3150 4050 50  0001 C CNN
 F 1 "GND" H 3150 4150 50  0000 C CNN
 F 2 "" H 3150 4300 50  0001 C CNN
@@
 	1750 1650 1750 2450
 $Comp
-L GND #PWR1
+L GND #PWR09
 U 1 1 5B7E721D
 P 1750 2450
-F 0 "#PWR1" H 1750 2200 50  0001 C CNN
+F 0 "#PWR09" H 1750 2200 50  0001 C CNN
 F 1 "GND" H 1750 2300 50  0000 C CNN
 F 2 "" H 1750 2450 50  0001 C CNN
@@
 $EndComp
 $Comp
-L GND #PWR7
+L GND #PWR010
 U 1 1 5B84307B
 P 5750 3550
-F 0 "#PWR7" H 5750 3300 50  0001 C CNN
+F 0 "#PWR010" H 5750 3300 50  0001 C CNN
 F 1 "GND" H 5750 3400 50  0000 C CNN
 F 2 "" H 5750 3550 50  0001 C CNN
@@
 Entry Wire Line
 	4700 3350 4800 3250
-$Comp
-L CP_Small C1
-U 1 1 5B843283
-P 5150 2800
-F 0 "C1" H 5160 2870 50  0000 L CNN
-F 1 "10mF" H 5160 2720 50  0000 L CNN
-F 2 "Capacitors_THT:CP_Radial_D5.0mm_P2.50mm" H 5150 2800 50  0001 C CNN
-F 3 "" H 5150 2800 50  0001 C CNN
-	1    5150 2800
-	0    -1   -1   0
-$EndComp
-$Comp
-L CP_Small C2
-U 1 1 5B843336
-P 5150 3250
-F 0 "C2" H 5160 3320 50  0000 L CNN
-F 1 "10mF" H 5160 3170 50  0000 L CNN
-F 2 "Capacitors_THT:CP_Radial_D5.0mm_P2.50mm" H 5150 3250 50  0001 C CNN
-F 3 "" H 5150 3250 50  0001 C CNN
-	1    5150 3250
-	0    -1   -1   0
-$EndComp
-Wire Wire Line
-	5250 2800 5300 2800
-Wire Wire Line
-	5050 2800 4800 2800
-Wire Wire Line
-	4800 3250 5050 3250
-Wire Wire Line
-	5250 3250 5300 3250
+Wire Wire Line
+	4800 2800 5300 2800
+Wire Wire Line
+	4800 3250 5300 3250
 Wire Wire Line
 	5300 2900 5300 3100
@@
 F 0 "SW1" H 6600 3600 50  0000 L CNN
 F 1 "Turn" H 6550 3440 50  0000 C CNN
-F 2 "Buttons_Switches_SMD:SW_SPST_PTS645" H 6550 3700 50  0001 C CNN
+F 2 "Buttons_Switches_THT:SW_PUSH_6mm_h8.5mm" H 6550 3700 50  0001 C CNN
 F 3 "" H 6550 3700 50  0001 C CNN
 	1    6550 3500
@@
 	6950 3500 6750 3500
 $Comp
-L +5V #PWR8
+L +5V #PWR011
 U 1 1 5B84FD26
 P 6200 3050
-F 0 "#PWR8" H 6200 2900 50  0001 C CNN
+F 0 "#PWR011" H 6200 2900 50  0001 C CNN
 F 1 "+5V" H 6200 3190 50  0000 C CNN
 F 2 "" H 6200 3050 50  0001 C CNN
@@
 Text Label 4250 2950 0    60   ~ 0
 m2a
-$Comp
-L AVR-ISP-6 CON2
-U 1 1 5B8636D0
-P 1250 5300
-F 0 "CON2" H 1145 5540 50  0000 C CNN
-F 1 "AVR-ISP-6" H 985 5070 50  0000 L BNN
-F 2 "Connectors:IDC_Header_Straight_6pins" V 730 5340 50  0001 C CNN
-F 3 "" H 1225 5300 50  0001 C CNN
-	1    1250 5300
-	1    0    0    -1
-$EndComp
-$Comp
-L GND #PWR3
-U 1 1 5B863C75
-P 1950 5500
-F 0 "#PWR3" H 1950 5250 50  0001 C CNN
-F 1 "GND" H 1950 5350 50  0000 C CNN
-F 2 "" H 1950 5500 50  0001 C CNN
-F 3 "" H 1950 5500 50  0001 C CNN
-	1    1950 5500
-	1    0    0    -1
-$EndComp
-$Comp
-L +5V #PWR2
-U 1 1 5B863EC4
-P 1950 5050
-F 0 "#PWR2" H 1950 4900 50  0001 C CNN
-F 1 "+5V" H 1950 5190 50  0000 C CNN
-F 2 "" H 1950 5050 50  0001 C CNN
-F 3 "" H 1950 5050 50  0001 C CNN
-	1    1950 5050
-	1    0    0    -1
-$EndComp
-Wire Wire Line
-	1350 5200 1950 5200
-Wire Wire Line
-	1950 5200 1950 5050
-Wire Wire Line
-	1350 5400 1950 5400
-Wire Wire Line
-	1950 5400 1950 5500
-Wire Wire Line
-	1350 5300 2250 5300
-Wire Wire Line
-	1100 5400 600  5400
-Wire Wire Line
-	1100 5300 600  5300
-Wire Wire Line
-	1100 5200 600  5200
-Text Label 1800 5300 0    60   ~ 0
-MOSI
-Text Label 650  5200 0    60   ~ 0
-MISO
-Text Label 650  5300 0    60   ~ 0
-SCK
-Text Label 650  5400 0    60   ~ 0
-RESET
 $EndSCHEMATC

Commit message: ;
Parts:
- added C1: 10m, Capacitors_THT:C_Disc_D3.8mm_W2.6mm_P2.50mm, symbol C_Small
Connections:
- wire segments 106 -> 108
Changed lines of the file:
@@
 	7300 2150 7300 2200
 $Comp
-L GND #PWR01
+L GND #PWR7
 U 1 1 5B7A7AAC
 P 6600 3050
-F 0 "#PWR01" H 6600 2800 50  0001 C CNN
+F 0 "#PWR7" H 6600 2800 50  0001 C CNN
 F 1 "GND" H 6600 2900 50  0000 C CNN
 F 2 "" H 6600 3050 50  0001 C CNN
@@
 Connection ~ 6650 2800
 $Comp
-L +12V #PWR02
+L +12V #PWR8
 U 1 1 5B7A7C3C
 P 7850 700
-F 0 "#PWR02" H 7850 550 50  0001 C CNN
+F 0 "#PWR8" H 7850 550 50  0001 C CNN
 F 1 "+12V" H 7850 840 50  0000 C CNN
 F 2 "" H 7850 700 50  0001 C CNN
@@
 $EndComp
 $Comp
-L +5V #PWR03
+L +5V #PWR3
 U 1 1 5B7A7CE0
 P 4550 650
-F 0 "#PWR03" H 4550 500 50  0001 C CNN
+F 0 "#PWR3" H 4550 500 50  0001 C CNN
 F 1 "+5V" H 4550 790 50  0000 C CNN
 F 2 "" H 4550 650 50  0001 C CNN
@@
 	1650 650  5200 650
 $Comp
-L GND #PWR04
+L GND #PWR4
 U 1 1 5B7A7EE1
 P 4850 750
-F 0 "#PWR04" H 4850 500 50  0001 C CNN
+F 0 "#PWR4" H 4850 500 50  0001 C CNN
 F 1 "GND" H 4850 600 50  0000 C CNN
 F 2 "" H 4850 750 50  0001 C CNN
@@
 $EndComp
 $Comp
-L GND #PWR05
+L GND #PWR10
 U 1 1 5B7A7EFE
 P 8150 800
-F 0 "#PWR05" H 8150 550 50  0001 C CNN
+F 0 "#PWR10" H 8150 550 50  0001 C CNN
 F 1 "GND" H 8150 650 50  0000 C CNN
 F 2 "" H 8150 800 50  0001 C CNN
@@
 $EndComp
 $Comp
-L +12V #PWR06
+L +12V #PWR9
 U 1 1 5B7C12D6
 P 8050 4750
-F 0 "#PWR06" H 8050 4600 50  0001 C CNN
+F 0 "#PWR9" H 8050 4600 50  0001 C CNN
 F 1 "+12V" H 8050 4890 50  0000 C CNN
 F 2 "" H 8050 4750 50  0001 C CNN
@@
 	8600 4950 8850 4950
 $Comp
-L GND #PWR07
+L GND #PWR11
 U 1 1 5B7C1985
 P 8600 5050
-F 0 "#PWR07" H 8600 4800 50  0001 C CNN
+F 0 "#PWR11" H 8600 4800 50  0001 C CNN
 F 1 "GND" H 8600 4900 50  0000 C CNN
 F 2 "" H 8600 5050 50  0001 C CNN
@@
 Connection ~ 4550 650
 $Comp
-L GND #PWR08
+L GND #PWR2
 U 1 1 5B7E4EA7
 P 3150 4300
-F 0 "#PWR08" H 3150 4050 50  0001 C CNN
+F 0 "#PWR2" H 3150 4050 50  0001 C CNN
 F 1 "GND" H 3150 4150 50  0000 C CNN
 F 2 "" H 3150 4300 50  0001 C CNN
@@
 	1750 1650 1750 2450
 $Comp
-L GND #PWR09
+L GND #PWR1
 U 1 1 5B7E721D
 P 1750 2450
-F 0 "#PWR09" H 1750 2200 50  0001 C CNN
+F 0 "#PWR1" H 1750 2200 50  0001 C CNN
 F 1 "GND" H 1750 2300 50  0000 C CNN
 F 2 "" H 1750 2450 50  0001 C CNN
@@
 $EndComp
 $Comp
-L GND #PWR010
+L GND #PWR5
 U 1 1 5B84307B
 P 5750 3550
-F 0 "#PWR010" H 5750 3300 50  0001 C CNN
+F 0 "#PWR5" H 5750 3300 50  0001 C CNN
 F 1 "GND" H 5750 3400 50  0000 C CNN
 F 2 "" H 5750 3550 50  0001 C CNN
@@
 	6950 3500 6750 3500
 $Comp
-L +5V #PWR011
+L +5V #PWR6
 U 1 1 5B84FD26
 P 6200 3050
-F 0 "#PWR011" H 6200 2900 50  0001 C CNN
+F 0 "#PWR6" H 6200 2900 50  0001 C CNN
 F 1 "+5V" H 6200 3190 50  0000 C CNN
 F 2 "" H 6200 3050 50  0001 C CNN
@@
 Text Label 4250 2950 0    60   ~ 0
 m2a
+$Comp
+L C_Small C1
+U 1 1 5B9F9468
+P 6700 3700
+F 0 "C1" H 6710 3770 50  0000 L CNN
+F 1 "10m" H 6710 3620 50  0000 L CNN
+F 2 "Capacitors_THT:C_Disc_D3.8mm_W2.6mm_P2.50mm" H 6700 3700 50  0001 C CNN
+F 3 "" H 6700 3700 50  0001 C CNN
+	1    6700 3700
+	0    1    1    0
+$EndComp
+Wire Wire Line
+	6800 3700 6800 3500
+Connection ~ 6800 3500
+Wire Wire Line
+	6600 3700 6200 3700
+Connection ~ 6200 3700
 $EndSCHEMATC

Commit message: up01
Connections:
- wire segments 108 -> 110
Changed lines of the file:
@@
 	6600 3700 6200 3700
 Connection ~ 6200 3700
+Wire Wire Line
+	2250 1550 2100 1550
+Wire Wire Line
+	2100 1550 2100 1450
+Connection ~ 2100 1450
 $EndSCHEMATC
