File: waterlock/tqfp.kicad_pcb (KiCad board)
At the start: 2 copper layers, 26 parts, among them CON1 AVR-ISP-10, J1 v5, J2 v12, J3 m1, J4 m2, J5 Battery, J6 L1, J7 L2, SW1 Turn, U1 ATMEGA8-16PU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

Commit message: newpcb
Parts:
- CON1: footprint Connectors:IDC_Header_Straight_10pins -> Pin_Headers:Pin_Header_Straight_1x06_Pitch2.54mm; moved to B.Cu
- moved CON1 17.0 mm to (66.7, 26.3), turned to 180 degrees
- moved BZ1 7.60 mm to (63.8, 68.5), turned to 180 degrees
- moved SW1 3.61 mm to (65.3, 55.7)
Connections:
- CON1 pad 1: /MOSI -> /RESET
- CON1 pad 2: +5V -> /SCK
- CON1 pad 3: Net-(CON1-Pad3) -> /MISO
- CON1 pad 4: GND -> /MOSI
- CON1 pad 5: /RESET -> +5V
Routing:
- net GND: track 5.11 -> 123.4 mm, vias 0 -> 6
- net /pwr_c2: track 3.49 -> 89.1 mm, vias 0 -> 2
- net +5V: track 81.0 -> 160.8 mm, vias 0 -> 2
- net /pwr_c1: track 3.65 -> 64.0 mm, vias 0 -> 2
- net /buzz: track 0.00 -> 46.4 mm
- net /btn_1: track 11.8 -> 40.1 mm
- net /RESET: track 3.03 -> 29.7 mm, vias 0 -> 1
- net /led2: track 0.00 -> 13.3 mm, vias 0 -> 1
- net /led1: track 0.00 -> 12.4 mm, vias 0 -> 1
- net /MOSI: track 0.00 -> 6.78 mm
- net /MISO: track 0.00 -> 5.69 mm
- net /SCK: track 0.00 -> 4.08 mm
- net Net-(D4-Pad1): track 0.00 -> 2.63 mm
- net Net-(D3-Pad1): track 0.00 -> 2.63 mm
- net Net-(D2-Pad2): track 18.9 -> 20.5 mm
- added copper zone on B.Cu, net GND
- added copper zone on F.Cu, net GND
Other:
- board outline added: 55.1 x 64.2 mm
