File: waterlock/ds1307.sch (KiCad schematic (older format))
At the start: 4 parts

Commit message: pcb-prod
Parts:
- gave numbers to parts that had none: 4
Changed lines of the file:
@@
 $Descr A4 11693 8268
 encoding utf-8
-Sheet 3 3
+Sheet 2 3
 Title ""
 Date ""
@@
 $EndDescr
 $Comp
-L DS1307+ U?
+L DS1307+ U2
 U 1 1 5C063A62
 P 3350 1900
-F 0 "U?" H 3620 2450 50  0000 C CNN
+F 0 "U2" H 3620 2450 50  0000 C CNN
 F 1 "DS1307+" H 3650 1350 50  0000 C CNN
 F 2 "Housings_SOIC:SOIC-8_3.9x4.9mm_Pitch1.27mm" H 3350 1900 50  0001 C CNN
@@
 rtc_sda
 $Comp
-L Crystal_Small Y?
+L Crystal_Small Y1
 U 1 1 5C063B90
 P 2400 2200
-F 0 "Y?" H 2400 2300 50  0000 C CNN
+F 0 "Y1" H 2400 2300 50  0000 C CNN
 F 1 "Crystal_Small" H 2400 2100 50  0000 C CNN
 F 2 "Crystals:Crystal_C38-LF_d3.0mm_l8.0mm_Horizontal_1EP_style2" H 2400 2200 50  0001 C CNN
@@
 rtc_bat
 $Comp
-L +5V #PWR?
+L +5V #PWR15
 U 1 1 5C063BFA
 P 3350 850
-F 0 "#PWR?" H 3350 700 50  0001 C CNN
+F 0 "#PWR15" H 3350 700 50  0001 C CNN
 F 1 "+5V" H 3350 990 50  0000 C CNN
 F 2 "" H 3350 850 50  0001 C CNN
@@
 $EndComp
 $Comp
-L GND #PWR?
+L GND #PWR14
 U 1 1 5C063C12
 P 3050 2950
-F 0 "#PWR?" H 3050 2700 50  0001 C CNN
+F 0 "#PWR14" H 3050 2700 50  0001 C CNN
 F 1 "GND" H 3050 2800 50  0000 C CNN
 F 2 "" H 3050 2950 50  0001 C CNN
@@
 	3350 850  3350 1300
 $Comp
-L D_ALT D?
+L D_ALT D5
 U 1 1 5C0696C4
 P 4150 2200
-F 0 "D?" H 4150 2300 50  0000 C CNN
+F 0 "D5" H 4150 2300 50  0000 C CNN
 F 1 "D_ALT" H 4150 2100 50  0000 C CNN
 F 2 "Diodes_SMD:D_SMA" H 4150 2200 50  0001 C CNN
@@
 $EndComp
 $Comp
-L D_ALT D?
+L D_ALT D6
 U 1 1 5C06971E
 P 4500 2200
-F 0 "D?" H 4500 2300 50  0000 C CNN
+F 0 "D6" H 4500 2300 50  0000 C CNN
 F 1 "D_ALT" H 4500 2100 50  0000 C CNN
 F 2 "Diodes_SMD:D_SMA" H 4500 2200 50  0001 C CNN
