File: waterlock/controllerTFQP.kicad_pcb (KiCad board)
At the start: 2 copper layers, 99 x 50 mm, 40 parts, among them J10 m1-sensor, J2 v12, J3 m1, J4 m2, J8 Conn_01x06, J9 m2-sensor, Q1 2SC1945, Q2 2SC1945, Q3 2SC1945, Q4 2SC1945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

Commit message: ddpcb+
Parts:
- added REF**: MountingHole_6.5mm, Mounting_Holes:MountingHole_6.5mm, F.Cu at (71.1, 21.6)
- moved D1 6.24 mm to (80.6, 27.9)
Routing:
- net /pwr_c2: track 19.8 -> 14.6 mm
- net +5V: track 241.7 -> 244.4 mm

Commit message: pcb-prod
Parts:
- removed J10: m1-sensor, Connectors_Terminal_Blocks:TerminalBlock_Pheonix_MKDS1.5-2pol
- removed J9: m2-sensor, Connectors_Terminal_Blocks:TerminalBlock_Pheonix_MKDS1.5-2pol
- removed Q1, Q2, Q3, Q4: 2SC1945, TO_SOT_Packages_SMD:TSOT-23
- removed R11, R12, R13, R14: 10k, Resistors_SMD:R_1206_HandSoldering
- removed R15, R16: 1k, Resistors_SMD:R_1206_HandSoldering
- removed Sens_1: L1, Connectors_Terminal_Blocks:TerminalBlock_Pheonix_MKDS1.5-2pol
- removed Sens_2: L2, Connectors_Terminal_Blocks:TerminalBlock_Pheonix_MKDS1.5-2pol
- added D5: D_ALT, Diodes_SMD:D_SMA, F.Cu at (115.1, 33.4)
- added D6: D_ALT, Diodes_SMD:D_SMA, F.Cu at (115.1, 29.5)
- added D7: D_Schottky, Diodes_THT:D_DO-15_P10.16mm_Horizontal, F.Cu at (42.4, 54.2)
- added D8: D_Schottky, Diodes_THT:D_DO-15_P10.16mm_Horizontal, F.Cu at (55.7, 43.8)
- added J6: L1, Connectors_Terminal_Blocks:TerminalBlock_Philmore_TB132_02x5mm_Straight, F.Cu at (99.1, 65.0)
- added J7: L2, Connectors_Terminal_Blocks:TerminalBlock_Philmore_TB132_02x5mm_Straight, F.Cu at (110.7, 64.9)
- added U2: DS1307+, Housings_SOIC:SOIC-8_3.9x4.9mm_Pitch1.27mm, F.Cu at (106.4, 37.3)
- added U4: PC817, Housings_DIP:DIP-4_W7.62mm, F.Cu at (25.1, 52.8)
- added U5: PC817, Housings_DIP:DIP-4_W7.62mm, F.Cu at (47.3, 53.3)
- added Y1: Crystal_Small, Crystals:Crystal_C38-LF_d3.0mm_l8.0mm_Horizontal_1EP_style2, F.Cu at (115.8, 38.7)
- J3, J4: footprint Connectors_Terminal_Blocks:TerminalBlock_Pheonix_MKDS1.5-2pol -> Connectors_Terminal_Blocks:TerminalBlock_Philmore_TB133_03x5mm_Straight
- R10, R7, R8, R9: footprint Resistors_SMD:R_1206_HandSoldering -> Resistors_SMD:R_0805_HandSoldering
- moved R3 71.6 mm to (108.1, 28.0), turned to 0 degrees
- moved R2 48.3 mm to (108.1, 31.1), turned to 0 degrees
- moved R7 40.5 mm to (24.6, 41.2), turned to 180 degrees
- moved R9 31.8 mm to (31.1, 58.6), turned to 180 degrees
- moved R8 24.0 mm to (61.3, 50.1), turned to 270 degrees
- moved R10 19.2 mm to (50.8, 58.4), turned to 180 degrees
- moved J3 10.1 mm to (35.7, 64.5)
- moved BZ1 9.55 mm to (104.7, 52.6)
- moved J4 4.46 mm to (52.2, 64.5)
Connections:
- net Net-(J3-Pad2) renamed /MotorsShield/m1black
- net Net-(J4-Pad2) renamed /MotorsShield/m2black
- R10 pad 1: /MISO -> /MotorsShield/m2sensor
- R10 pad 2: +5V -> Net-(R10-Pad2)
- R2 pad 1: Net-(Q1-Pad1) -> /SDA
- R2 pad 2: /Postion_control/Left_pos_sens_1 -> +5V
- R3 pad 1: Net-(Q2-Pad1) -> /SCL
- R3 pad 2: /Postion_control/Left_pos_sens_2 -> +5V
- R7 pad 1: GND -> /SCK
- R7 pad 2: Net-(Q1-Pad1) -> +5V
- R8 pad 1: GND -> /MISO
- R8 pad 2: Net-(Q2-Pad1) -> +5V
- R9 pad 1: /SS -> /MotorsShield/m1sensor
- R9 pad 2: +5V -> Net-(R9-Pad2)
- U1 pad 27: Net-(U1-Pad27) -> /SDA
- U1 pad 28: Net-(U1-Pad28) -> /SCL
Routing:
- net /MOSI: track 72.2 -> 25.8 mm, vias 2 -> 0
- net /SCL: track 0.00 -> 46.0 mm, vias 0 -> 2
- net +5V: track 244.4 -> 286.3 mm
- net /SDA: track 0.00 -> 36.7 mm, vias 0 -> 2
- net /MotorsShield/m1sensor: track 0.00 -> 25.9 mm
- net /SS: track 24.3 -> 0.16 mm, vias 2 -> 0
- net /MotorsShield/m2black: track 51.1 -> 69.6 mm
- net Net-(J4-Pad1): track 29.8 -> 46.8 mm
- net /pwr_c1: track 38.6 -> 53.4 mm
- net /MotorsShield/m2sensor: track 0.00 -> 13.6 mm
- net /SCK: track 79.6 -> 92.1 mm
- net Net-(U2-Pad2): track 0.00 -> 11.4 mm
- net /Postion_control/Right_pos_sens_1: track 10.4 -> 0.00 mm
- net /Postion_control/Right_pos_sens_2: track 9.33 -> 0.00 mm
- net /buzz: track 74.3 -> 65.0 mm
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
Commit message: pcb-prod
Parts:
- moved REF** 0.90 mm to (70.5, 21.0)
Routing:
- net /SCL: track 46.0 -> 46.6 mm
Changed lines of the file:
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@@
     (links 88)
     (no_connects 0)
-    (area 20.949999 13.115 120.8842 72.9482)
+    (area 20.949999 13.115 120.091201 72.491)
     (thickness 1.6)
     (drawings 14)
-    (tracks 407)
+    (tracks 410)
     (zones 0)
     (modules 37)
@@
   (page A4)
   (layers
-    (0 F.Cu signal)
-    (31 B.Cu signal)
-    (32 B.Adhes user)
-    (33 F.Adhes user)
+    (0 F.Cu signal hide)
+    (31 B.Cu signal hide)
+    (32 B.Adhes user hide)
+    (33 F.Adhes user hide)
     (34 B.Paste user)
     (35 F.Paste user)
@@
   )
   (setup
-    (last_trace_width 0.6096)
+    (last_trace_width 0.3048)
     (user_trace_width 0.1524)
     (user_trace_width 0.3048)
@@
   )
   (module Mounting_Holes:MountingHole_6.5mm (layer F.Cu)
-    (at 71.12 21.59)
+    (at 70.4596 20.9804)
     (descr "Mounting Hole 6.5mm, no annular")
     (tags "mounting hole 6.5mm no annular")
@@
       (effects (font (size 1 1) (thickness 0.15)))
     )
-    (fp_text value MountingHole_6.5mm (at 0 7.5) (layer F.Fab)
+    (fp_text value MountingHole_6.5mm (at 0.0508 0.3556) (layer F.Fab)
       (effects (font (size 1 1) (thickness 0.15)))
     )
@@
     (descr "D, DO-15 series, Axial, Horizontal, pin pitch=10.16mm, , length*diameter=7.6*3.6mm^2, , http://www.diodes.com/_files/packages/DO-15.pdf")
     (tags "D DO-15 series Axial Horizontal pin pitch 10.16mm  length 7.6mm diameter 3.6mm")
-    (fp_text reference D7 (at 5.08 -2.86 180) (layer F.SilkS)
-      (effects (font (size 1 1) (thickness 0.15)))
-    )
-    (fp_text value D_Schottky (at 5.08 2.86 180) (layer F.Fab)
-      (effects (font (size 1 1) (thickness 0.15)))
-    )
-    (fp_text user %R (at 5.08 0.1524 180) (layer F.Fab)
+    (fp_text reference D7 (at 4.9276 3.048 180) (layer F.SilkS)
+      (effects (font (size 1 1) (thickness 0.15)))
+    )
+    (fp_text value D_Schottky (at 4.7244 1.3716 180) (layer F.Fab)
+      (effects (font (size 1 1) (thickness 0.15)))
+    )
+    (fp_text user %R (at 4.9784 2.8956 180) (layer F.Fab)
       (effects (font (size 1 1) (thickness 0.15)))
     )
@@
     (descr "3-way 5.0mm pitch terminal block, http://www.philmore-datak.com/mc/Page%20197.pdf")
     (tags "screw terminal block")
-    (fp_text reference J3 (at 5 -6) (layer F.SilkS)
+    (fp_text reference J3 (at 4.92 -5.6388) (layer F.SilkS)
       (effects (font (size 1 1) (thickness 0.15)))
     )
@@
       (effects (font (size 1 1) (thickness 0.15)))
     )
-    (fp_text value L1 (at 2.5 6.9) (layer F.Fab)
+    (fp_text value L1 (at 2.46 4.7244) (layer F.Fab)
       (effects (font (size 1 1) (thickness 0.15)))
     )
@@
       (effects (font (size 1 1) (thickness 0.15)))
     )
-    (fp_text value L2 (at 2.5 6.9) (layer F.Fab)
+    (fp_text value L2 (at 2.6924 4.9784) (layer F.Fab)
       (effects (font (size 1 1) (thickness 0.15)))
     )
@@
       (effects (font (size 1 1) (thickness 0.15)))
     )
-    (fp_text user %R (at 3.81 1.27 90) (layer F.Fab)
+    (fp_text user %R (at 3.8608 1.27 90) (layer F.Fab)
       (effects (font (size 1 1) (thickness 0.15)))
     )
@@
       (effects (font (size 1 1) (thickness 0.15)))
     )
-    (fp_text value Crystal_Small (at 3.97 2.25 90) (layer F.Fab)
+    (fp_text value Crystal_Small (at 1.0008 6.5428 90) (layer F.Fab)
       (effects (font (size 1 1) (thickness 0.15)))
     )
@@
     )
   )
-  (dimension 50.165 (width 0.3) (layer Dwgs.User)
-    (gr_text "50,165 мм" (at 46.0375 17.7) (layer Dwgs.User)
+  (dimension 49.504704 (width 0.3) (layer Dwgs.User)
+    (gr_text "49,505 mm" (at 45.70161 17.496806 0.1175899416) (layer Dwgs.User)
       (effects (font (size 1.5 1.5) (thickness 0.3)))
     )
-    (feature1 (pts (xy 71.12 20.32) (xy 71.12 16.35)))
-    (feature2 (pts (xy 20.955 20.32) (xy 20.955 16.35)))
-    (crossbar (pts (xy 20.955 19.05) (xy 71.12 19.05)))
-    (arrow1a (pts (xy 71.12 19.05) (xy 69.993496 19.636421)))
-    (arrow1b (pts (xy 71.12 19.05) (xy 69.993496 18.463579)))
-    (arrow2a (pts (xy 20.955 19.05) (xy 22.081504 19.636421)))
-    (arrow2b (pts (xy 20.955 19.05) (xy 22.081504 18.463579)))
+    (feature1 (pts (xy 70.4596 20.2184) (xy 70.45114 16.096009)))
+    (feature2 (pts (xy 20.955 20.32) (xy 20.94654 16.197609)))
+    (crossbar (pts (xy 20.952081 18.897603) (xy 70.456681 18.796003)))
+    (arrow1a (pts (xy 70.456681 18.796003) (xy 69.331383 19.384734)))
+    (arrow1b (pts (xy 70.456681 18.796003) (xy 69.328976 18.211895)))
+    (arrow2a (pts (xy 20.952081 18.897603) (xy 22.079786 19.481711)))
+    (arrow2b (pts (xy 20.952081 18.897603) (xy 22.077379 18.308872)))
   )
   (dimension 99.06 (width 0.3) (layer Dwgs.User)
@@
   (segment (start 62.23 64.516) (end 62.23 62.818944) (width 0.8128) (layer F.Cu) (net 36))
   (segment (start 62.23 62.818944) (end 59.69 60.278944) (width 0.8128) (layer F.Cu) (net 36))
+  (segment (start 106.0836 31.0896) (end 105.9336 31.0896) (width 0.3048) (layer F.Cu) (net 37))
+  (segment (start 105.9336 31.0896) (end 103.726 33.2972) (width 0.3048) (layer F.Cu) (net 37))
+  (segment (start 103.726 33.2972) (end 103.726 35.433) (width 0.3048) (layer F.Cu) (net 37))
   (segment (start 85.2932 33.3756) (end 85.593199 33.075601) (width 0.3048) (layer F.Cu) (net 37))
   (segment (start 85.593199 33.075601) (end 85.593199 33.024447) (width 0.3048) (layer F.Cu) (net 37))
@@
   (segment (start 80.0224 32.0424) (end 80.1624 31.9024) (width 0.3048) (layer F.Cu) (net 37))
   (via (at 80.1624 31.9024) (size 0.6) (drill 0.4) (layers F.Cu B.Cu) (net 37))
-  (segment (start 106.0836 31.0896) (end 106.0836 33.5504) (width 0.3048) (layer F.Cu) (net 37))
-  (segment (start 106.0836 33.5504) (end 104.201 35.433) (width 0.3048) (layer F.Cu) (net 37))
-  (segment (start 104.201 35.433) (end 103.726 35.433) (width 0.3048) (layer F.Cu) (net 37))
+  (segment (start 108.1532 32.0548) (end 108.1532 28.7556) (width 0.3048) (layer F.Cu) (net 38))
+  (segment (start 108.1532 28.7556) (end 107.4392 28.0416) (width 0.3048) (layer F.Cu) (net 38))
+  (segment (start 107.5436 32.6644) (end 108.1532 32.0548) (width 0.3048) (layer F.Cu) (net 38))
+  (segment (start 107.4928 32.6644) (end 107.5436 32.6644) (width 0.3048) (layer F.Cu) (net 38))
+  (segment (start 103.726 36.703) (end 104.8258 36.703) (width 0.3048) (layer F.Cu) (net 38))
+  (segment (start 106.0196 35.5092) (end 106.0196 34.1376) (width 0.3048) (layer F.Cu) (net 38))
+  (segment (start 107.4392 28.0416) (end 106.1344 28.0416) (width 0.3048) (layer F.Cu) (net 38))
+  (segment (start 104.8258 36.703) (end 106.0196 35.5092) (width 0.3048) (layer F.Cu) (net 38))
+  (segment (start 106.0196 34.1376) (end 107.4928 32.6644) (width 0.3048) (layer F.Cu) (net 38))
   (segment (start 79.2988 30.7848) (end 79.2988 36.9404) (width 0.3048) (layer F.Cu) (net 38))
   (segment (start 79.2988 36.9404) (end 79.2224 37.0168) (width 0.3048) (layer F.Cu) (net 38))
@@
   (segment (start 79.248 36.9912) (end 79.2224 37.0168) (width 0.3048) (layer F.Cu) (net 38))
   (segment (start 103.726 36.703) (end 103.251 36.703) (width 0.3048) (layer F.Cu) (net 38))
-  (segment (start 106.1344 28.0416) (end 107.4392 28.0416) (width 0.3048) (layer F.Cu) (net 38))
-  (segment (start 107.4392 28.0416) (end 107.4928 28.0952) (width 0.3048) (layer F.Cu) (net 38))
-  (segment (start 107.4928 28.0952) (end 107.4928 34.036) (width 0.3048) (layer F.Cu) (net 38))
-  (segment (start 104.8004 36.703) (end 103.726 36.703) (width 0.3048) (layer F.Cu) (net 38))
-  (segment (start 107.4928 34.036) (end 104.8258 36.703) (width 0.3048) (layer F.Cu) (net 38))
-  (segment (start 104.8258 36.703) (end 104.8004 36.703) (width 0.3048) (layer F.Cu) (net 38))
   (segment (start 29.7396 58.6232) (end 28.38 58.6232) (width 0.6096) (layer F.Cu) (net 39))
   (segment (start 28.38 58.6232) (end 25.0952 55.3384) (width 0.6096) (layer F.Cu) (net 39))
@@
       )
     )
+  )
+  (zone (net 0) (net_name "") (layer F.Cu) (hatch edge 0.508)
+    (connect_pads (clearance 0.508))
+    (min_thickness 0.254)
+    (keepout (tracks allowed) (vias allowed) (copperpour not_allowed))
+    (fill yes (arc_segments 16) (thermal_gap 0.508) (thermal_bridge_width 0.508))
+    (polygon
+      (pts
+        (xy 115.2144 26.3652) (xy 119.2276 26.416) (xy 119.2276 35.2044) (xy 111.0488 35.2044) (xy 111.0488 26.2636)
+      )
+    )
+  )
+  (zone (net 0) (net_name "") (layer B.Cu) (hatch edge 0.508)
+    (connect_pads (clearance 0.508))
+    (min_thickness 0.254)
+    (keepout (tracks allowed) (vias allowed) (copperpour not_allowed))
+    (fill yes (arc_segments 16) (thermal_gap 0.508) (thermal_bridge_width 0.508))
+    (polygon
+      (pts
+        (xy 112.268 35.56) (xy 118.9228 35.56) (xy 118.9228 40.132) (xy 112.268 40.1828)
+      )
+    )

Commit message: input 5v
Parts:
- added 5out: SolderWirePad_2x_2mmDrill, Wire_Pads:SolderWirePad_2x_2mmDrill, F.Cu at (83.5, 23.5)
- moved VCC 9.00 mm to (92.5, 23.5)
- moved BAT 6.15 mm to (106.8, 23.7)
Routing:
- net /pwr_c2: track 14.6 -> 21.6 mm
- net /pwr_c1: track 53.4 -> 47.8 mm
- net +5V: track 286.3 -> 291.0 mm

Commit message: prod
Parts:
- D1: value 1N -> SS16
- D7, D8: value D_Schottky -> 1N5822
- J3: value m1 -> 300-031-7,5
- J4: value m2 -> 300-031-7,5
- J6: value L1 -> 301-021-12
- J7: value L2 -> 301-021-12
- SW1: value Turn -> Tactile Angle
- Y1: value Crystal_Small -> 32768Hz
Changed lines of the file:
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@@
-(kicad_pcb (version 4) (host pcbnew 4.0.4-snap1-stable)
+(kicad_pcb (version 4) (host pcbnew 4.0.7-e2-6376~61~ubuntu18.04.1)
   (general
     (links 90)
     (no_connects 0)
-    (area 20.94654 12.5054 120.091201 72.491)
+    (area 20.94654 12.5054 121.276701 72.491)
     (thickness 1.6)
     (drawings 14)
@@
   (layers
     (0 F.Cu signal hide)
-    (31 B.Cu signal)
+    (31 B.Cu signal hide)
     (32 B.Adhes user)
     (33 F.Adhes user)
@@
   )
   (setup
-    (last_trace_width 0.8128)
+    (last_trace_width 0.25)
     (user_trace_width 0.1524)
     (user_trace_width 0.3048)
@@
       (effects (font (size 1 1) (thickness 0.15)))
     )
-    (fp_text value 1N (at 0 2.6) (layer F.Fab)
+    (fp_text value SS16 (at 0 2.6) (layer F.Fab)
       (effects (font (size 1 1) (thickness 0.15)))
     )
@@
       (effects (font (size 1 1) (thickness 0.15)))
     )
-    (fp_text value Turn (at 2.25 5.38988 180) (layer F.Fab)
+    (fp_text value "Tactile Angle" (at 2.25 5.38988 180) (layer F.Fab)
       (effects (font (size 1 1) (thickness 0.15)))
     )
@@
       (effects (font (size 1 1) (thickness 0.15)))
     )
-    (fp_text value D_Schottky (at 4.7244 1.3716 180) (layer F.Fab)
+    (fp_text value 1N5822 (at 4.7244 1.3716 180) (layer F.Fab)
       (effects (font (size 1 1) (thickness 0.15)))
     )
@@
       (effects (font (size 1 1) (thickness 0.15)))
     )
-    (fp_text value D_Schottky (at 5.08 2.86 270) (layer F.Fab)
+    (fp_text value 1N5822 (at 5.08 2.86 270) (layer F.Fab)
       (effects (font (size 1 1) (thickness 0.15)))
     )
@@
       (effects (font (size 1 1) (thickness 0.15)))
     )
-    (fp_text value m1 (at 5 6.9) (layer F.Fab)
+    (fp_text value 300-031-7,5 (at 5 6.9) (layer F.Fab)
       (effects (font (size 1 1) (thickness 0.15)))
     )
@@
       (effects (font (size 1 1) (thickness 0.15)))
     )
-    (fp_text value m2 (at 5 6.9) (layer F.Fab)
+    (fp_text value 300-031-7,5 (at 5 6.9) (layer F.Fab)
       (effects (font (size 1 1) (thickness 0.15)))
     )
@@
       (effects (font (size 1 1) (thickness 0.15)))
     )
-    (fp_text value L1 (at 2.46 4.7244) (layer F.Fab)
+    (fp_text value 301-021-12 (at 2.46 4.7244) (layer F.Fab)
       (effects (font (size 1 1) (thickness 0.15)))
     )
@@
       (effects (font (size 1 1) (thickness 0.15)))
     )
-    (fp_text value L2 (at 2.6924 4.9784) (layer F.Fab)
+    (fp_text value 301-021-12 (at 2.6924 4.9784) (layer F.Fab)
       (effects (font (size 1 1) (thickness 0.15)))
     )
@@
       (effects (font (size 1 1) (thickness 0.15)))
     )
-    (fp_text value Crystal_Small (at 1.0008 6.5428 90) (layer F.Fab)
-      (effects (font (size 1 1) (thickness 0.15)))
-    )
+    (fp_text value 32768Hz (at 1.0008 6.5428 90) (layer F.Fab)
+      (effects (font (size 1 1) (thickness 0.15)))
+    )
