File: waterlock/controllerTFQP.sch (KiCad schematic (older format))
At the start: 27 parts, among them J1 v5, J2 v12, J3 m1, J4 m2, J5 Battery, J6 L1, J7 L2, SW1 Turn, U1 ATMEGA8-16PU, U2 LM317_3PinPackage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

Commit message: newpcb
Parts:
- C1, C3: footprint Capacitors_THT:C_Disc_D3.8mm_W2.6mm_P2.50mm -> Capacitors_SMD:C_1206_HandSoldering
- J2: footprint Connectors_Terminal_Blocks:TerminalBlock_Philmore_TB132_02x5mm_Straight -> Connectors:JACK_ALIM
- R1, R2, R3, R4, R5, R6, R7, R8: footprint Resistors_THT:R_Axial_DIN0207_L6.3mm_D2.5mm_P7.62mm_Horizontal -> Resistors_SMD:R_1206_HandSoldering
- SW1: footprint Buttons_Switches_THT:SW_PUSH_6mm_h8.5mm -> Buttons_Switches_THT:SW_Tactile_SPST_Angled_PTS645Vx39-2LFS
- U1: footprint Housings_DIP:DIP-28_W7.62mm_LongPads -> Housings_QFP:TQFP-32_7x7mm_Pitch0.8mm
Changed lines of the file:
@@
 LIBS:contrib
 LIBS:valves
-LIBS:motor_drivers
-LIBS:controller-cache
+LIBS:controllerTFQP-cache
 EELAYER 25 0
 EELAYER END
@@
 F 0 "U1" H 2400 3650 50  0000 L BNN
 F 1 "ATMEGA8-16PU" H 3650 900 50  0000 L BNN
-F 2 "Housings_DIP:DIP-28_W7.62mm_LongPads" H 3150 2350 50  0001 C CIN
+F 2 "Housings_QFP:TQFP-32_7x7mm_Pitch0.8mm" H 3150 2350 50  0001 C CIN
 F 3 "" H 3150 2350 50  0001 C CNN
 	1    3150 2350
@@
 F 0 "J2" H 9050 800 50  0000 C CNN
 F 1 "v12" H 9050 500 50  0000 C CNN
-F 2 "Connectors_Terminal_Blocks:TerminalBlock_Philmore_TB132_02x5mm_Straight" H 9050 700 50  0001 C CNN
+F 2 "Connectors:JACK_ALIM" H 9050 700 50  0001 C CNN
 F 3 "" H 9050 700 50  0001 C CNN
 	1    9050 700
@@
 F 0 "R1" V 1930 1000 50  0000 C CNN
 F 1 "10k" V 1850 1000 50  0000 C CNN
-F 2 "Resistors_THT:R_Axial_DIN0207_L6.3mm_D2.5mm_P7.62mm_Horizontal" V 1780 1000 50  0001 C CNN
+F 2 "Resistors_SMD:R_1206_HandSoldering" V 1780 1000 50  0001 C CNN
 F 3 "" H 1850 1000 50  0001 C CNN
 	1    1850 1000
@@
 F 0 "R7" V 8780 4600 50  0000 C CNN
 F 1 "47k" V 8700 4600 50  0000 C CNN
-F 2 "Resistors_THT:R_Axial_DIN0207_L6.3mm_D2.5mm_P7.62mm_Horizontal" V 8630 4600 50  0001 C CNN
+F 2 "Resistors_SMD:R_1206_HandSoldering" V 8630 4600 50  0001 C CNN
 F 3 "" H 8700 4600 50  0001 C CNN
 	1    8700 4600
@@
 F 0 "R8" V 9180 4600 50  0000 C CNN
 F 1 "68k" V 9100 4600 50  0000 C CNN
-F 2 "Resistors_THT:R_Axial_DIN0207_L6.3mm_D2.5mm_P7.62mm_Horizontal" V 9030 4600 50  0001 C CNN
+F 2 "Resistors_SMD:R_1206_HandSoldering" V 9030 4600 50  0001 C CNN
 F 3 "" H 9100 4600 50  0001 C CNN
 	1    9100 4600
@@
 F 0 "R2" V 4730 4700 50  0000 C CNN
 F 1 "47k" V 4650 4700 50  0000 C CNN
-F 2 "Resistors_THT:R_Axial_DIN0207_L6.3mm_D2.5mm_P7.62mm_Horizontal" V 4580 4700 50  0001 C CNN
+F 2 "Resistors_SMD:R_1206_HandSoldering" V 4580 4700 50  0001 C CNN
 F 3 "" H 4650 4700 50  0001 C CNN
 	1    4650 4700
@@
 F 0 "R3" V 5280 4700 50  0000 C CNN
 F 1 "68k" V 5200 4700 50  0000 C CNN
-F 2 "Resistors_THT:R_Axial_DIN0207_L6.3mm_D2.5mm_P7.62mm_Horizontal" V 5130 4700 50  0001 C CNN
+F 2 "Resistors_SMD:R_1206_HandSoldering" V 5130 4700 50  0001 C CNN
 F 3 "" H 5200 4700 50  0001 C CNN
 	1    5200 4700
@@
 F 0 "SW1" H 6600 3600 50  0000 L CNN
 F 1 "Turn" H 6550 3440 50  0000 C CNN
-F 2 "Buttons_Switches_THT:SW_PUSH_6mm_h8.5mm" H 6550 3700 50  0001 C CNN
+F 2 "Buttons_Switches_THT:SW_Tactile_SPST_Angled_PTS645Vx39-2LFS" H 6550 3700 50  0001 C CNN
 F 3 "" H 6550 3700 50  0001 C CNN
 	1    6550 3500
@@
 F 0 "R5" V 7530 4700 50  0000 C CNN
 F 1 "10k" V 7450 4700 50  0000 C CNN
-F 2 "Resistors_THT:R_Axial_DIN0207_L6.3mm_D2.5mm_P7.62mm_Horizontal" V 7380 4700 50  0001 C CNN
+F 2 "Resistors_SMD:R_1206_HandSoldering" V 7380 4700 50  0001 C CNN
 F 3 "" H 7450 4700 50  0001 C CNN
 	1    7450 4700
@@
 F 0 "R6" V 7880 4700 50  0000 C CNN
 F 1 "10k" V 7800 4700 50  0000 C CNN
-F 2 "Resistors_THT:R_Axial_DIN0207_L6.3mm_D2.5mm_P7.62mm_Horizontal" V 7730 4700 50  0001 C CNN
+F 2 "Resistors_SMD:R_1206_HandSoldering" V 7730 4700 50  0001 C CNN
 F 3 "" H 7800 4700 50  0001 C CNN
 	1    7800 4700
@@
 F 0 "R4" V 6280 3300 50  0000 C CNN
 F 1 "10k" V 6200 3300 50  0000 C CNN
-F 2 "Resistors_THT:R_Axial_DIN0207_L6.3mm_D2.5mm_P7.62mm_Horizontal" V 6130 3300 50  0001 C CNN
+F 2 "Resistors_SMD:R_1206_HandSoldering" V 6130 3300 50  0001 C CNN
 F 3 "" H 6200 3300 50  0001 C CNN
 	1    6200 3300
@@
 F 0 "C3" H 1810 1520 50  0000 L CNN
 F 1 "10m" H 1810 1370 50  0000 L CNN
-F 2 "Capacitors_THT:C_Disc_D3.8mm_W2.6mm_P2.50mm" H 1800 1450 50  0001 C CNN
+F 2 "Capacitors_SMD:C_1206_HandSoldering" H 1800 1450 50  0001 C CNN
 F 3 "" H 1800 1450 50  0001 C CNN
 	1    1800 1450
@@
 F 0 "C1" H 6710 3770 50  0000 L CNN
 F 1 "10m" H 6710 3620 50  0000 L CNN
-F 2 "Capacitors_THT:C_Disc_D3.8mm_W2.6mm_P2.50mm" H 6700 3700 50  0001 C CNN
+F 2 "Capacitors_SMD:C_1206_HandSoldering" H 6700 3700 50  0001 C CNN
 F 3 "" H 6700 3700 50  0001 C CNN
 	1    6700 3700

Commit message: tqfp
Parts:
- removed R2, R7: 47k, Resistors_SMD:R_1206_HandSoldering, symbol R
- removed R3, R8: 68k, Resistors_SMD:R_1206_HandSoldering, symbol R
- removed U2: LM317_3PinPackage, symbol LM317_3PinPackage
- added J10: m1-sensor, Connectors_Terminal_Blocks:TerminalBlock_Philmore_TB132_02x5mm_Straight, symbol Conn_01x02
- added J9: m2-sensor, Connectors_Terminal_Blocks:TerminalBlock_Philmore_TB132_02x5mm_Straight, symbol Conn_01x02
- D1, D2: footprint Diodes_THT:D_DO-41_SOD81_P7.62mm_Horizontal -> Diodes_SMD:D_SMA_Handsoldering
- J2: footprint Connectors:JACK_ALIM -> Connectors_Terminal_Blocks:TerminalBlock_Philmore_TB132_02x5mm_Straight
- gave numbers to parts that had none: 1
Connections:
- net labels added: SS
- net labels removed: +12V, acdc_pwr
- wire segments 110 -> 120
Other:
- moved on the sheet: J1

Commit message: new wave
Parts:
- added R? (x2): 10k, Resistors_SMD:R_1206_HandSoldering, symbol R
Connections:
- net labels added: SCL, SDA
- wire segments 120 -> 132
Changed lines of the file:
@@
 LIBS:contrib
 LIBS:valves
+LIBS:maxim
 LIBS:controllerTFQP-cache
 EELAYER 25 0
@@
 $Descr A4 11693 8268
 encoding utf-8
-Sheet 1 2
+Sheet 1 3
 Title "Water leak protection"
 Date ""
@@
 Text Label 6200 4200 0    60   ~ 0
 pwr_c2
+$Sheet
+S 3350 5100 1200 1100
+U 5C0639DA
+F0 "RTC_ds1307" 60
+F1 "ds1307.sch" 60
+F2 "rtc_scl" I L 3350 5300 60
+F3 "rtc_sda" I L 3350 5500 60
+F4 "rtc_bat" I L 3350 5700 60
+$EndSheet
+Entry Wire Line
+	2250 3900 2350 4000
+Entry Wire Line
+	2550 3900 2650 4000
+Entry Wire Line
+	2850 3900 2950 4000
+Entry Wire Line
+	4600 2350 4700 2250
+Entry Wire Line
+	4600 2450 4700 2350
+Wire Wire Line
+	4150 2350 4600 2350
+Wire Wire Line
+	4150 2450 4600 2450
+Text Label 4250 2350 0    60   ~ 0
+SDA
+Text Label 4250 2450 0    60   ~ 0
+SCL
+$Comp
+L +5V #PWR?
+U 1 1 5C06FAFE
+P 1550 4250
+F 0 "#PWR?" H 1550 4100 50  0001 C CNN
+F 1 "+5V" H 1550 4390 50  0000 C CNN
+F 2 "" H 1550 4250 50  0001 C CNN
+F 3 "" H 1550 4250 50  0001 C CNN
+	1    1550 4250
+	1    0    0    -1
+$EndComp
+$Comp
+L R R?
+U 1 1 5C06FB93
+P 1800 4250
+F 0 "R?" V 1880 4250 50  0000 C CNN
+F 1 "10k" V 1800 4250 50  0000 C CNN
+F 2 "Resistors_SMD:R_1206_HandSoldering" V 1730 4250 50  0001 C CNN
+F 3 "" H 1800 4250 50  0001 C CNN
+	1    1800 4250
+	0    1    1    0
+$EndComp
+$Comp
+L R R?
+U 1 1 5C06FDBF
+P 1800 4500
+F 0 "R?" V 1880 4500 50  0000 C CNN
+F 1 "10k" V 1800 4500 50  0000 C CNN
+F 2 "Resistors_SMD:R_1206_HandSoldering" V 1730 4500 50  0001 C CNN
+F 3 "" H 1800 4500 50  0001 C CNN
+	1    1800 4500
+	0    1    1    0
+$EndComp
+Wire Wire Line
+	2950 4000 2950 5300
+Wire Wire Line
+	2950 5300 3350 5300
+Wire Wire Line
+	2650 4000 2650 5500
+Wire Wire Line
+	2650 5500 3350 5500
+Wire Wire Line
+	1550 4250 1650 4250
+Wire Wire Line
+	1650 4250 1650 4500
+Wire Wire Line
+	1950 4250 2650 4250
+Connection ~ 2650 4250
+Wire Wire Line
+	1950 4500 2950 4500
+Connection ~ 2950 4500
+Text Label 3050 5300 0    60   ~ 0
+SCL
+Text Label 3050 5500 0    60   ~ 0
+SDA
+Wire Wire Line
+	2350 4000 2350 5700
+Wire Wire Line
+	2350 5700 3350 5700
+Text Label 2900 5700 0    60   ~ 0
+pwr_c1
 $EndSCHEMATC

Commit message: pcb-prod
Parts:
- removed J10: m1-sensor, Connectors_Terminal_Blocks:TerminalBlock_Philmore_TB132_02x5mm_Straight, symbol Conn_01x02
- removed J3: m1, Connectors_Terminal_Blocks:TerminalBlock_Philmore_TB132_02x5mm_Straight, symbol Conn_01x02
- removed J4: m2, Connectors_Terminal_Blocks:TerminalBlock_Philmore_TB132_02x5mm_Straight, symbol Conn_01x02
- removed J9: m2-sensor, Connectors_Terminal_Blocks:TerminalBlock_Philmore_TB132_02x5mm_Straight, symbol Conn_01x02
- added J3: m1, Connectors_Terminal_Blocks:TerminalBlock_Philmore_TB133_03x5mm_Straight, symbol Conn_01x03
- added J4: m2, Connectors_Terminal_Blocks:TerminalBlock_Philmore_TB133_03x5mm_Straight, symbol Conn_01x03
- gave numbers to parts that had none: 2
Connections:
- wire segments 132 -> 145
Changed lines of the file:
@@
-$EndComp
-$Comp
-L Conn_01x02 J3
-U 1 1 5B7A7357
-P 8600 1300
-F 0 "J3" H 8600 1400 50  0000 C CNN
-F 1 "m1" H 8600 1100 50  0000 C CNN
-F 2 "Connectors_Terminal_Blocks:TerminalBlock_Philmore_TB132_02x5mm_Straight" H 8600 1300 50  0001 C CNN
-F 3 "" H 8600 1300 50  0001 C CNN
-	1    8600 1300
-	1    0    0    -1
-$EndComp
-$Comp
-L Conn_01x02 J4
-U 1 1 5B7A7664
-P 8600 2050
-F 0 "J4" H 8600 2150 50  0000 C CNN
-F 1 "m2" H 8600 1850 50  0000 C CNN
-F 2 "Connectors_Terminal_Blocks:TerminalBlock_Philmore_TB132_02x5mm_Straight" H 8600 2050 50  0001 C CNN
-F 3 "" H 8600 2050 50  0001 C CNN
-	1    8600 2050
-	1    0    0    -1
 $EndComp
 $Comp
@@
 	8000 1400 8000 1300
 Wire Wire Line
-	8000 1300 8400 1300
-Wire Wire Line
-	8400 1400 8150 1400
+	8000 1300 8600 1300
+Wire Wire Line
+	8150 1400 8600 1400
 Wire Wire Line
 	8150 1400 8150 1600
@@
 	8150 1600 7300 1600
 Wire Wire Line
-	7300 2000 8400 2000
-Wire Wire Line
-	8400 2000 8400 2050
-Wire Wire Line
-	8400 2150 7300 2150
+	7300 2000 8600 2000
+Wire Wire Line
+	7300 2150 8450 2150
 Wire Wire Line
 	7300 2150 7300 2200
 $Comp
-L GND #PWR01
+L GND #PWR8
 U 1 1 5B7A7AAC
 P 6600 3050
-F 0 "#PWR01" H 6600 2800 50  0001 C CNN
+F 0 "#PWR8" H 6600 2800 50  0001 C CNN
 F 1 "GND" H 6600 2900 50  0000 C CNN
 F 2 "" H 6600 3050 50  0001 C CNN
@@
 Connection ~ 6650 2800
 $Comp
-L +5V #PWR02
+L +5V #PWR4
 U 1 1 5B7A7CE0
 P 4550 650
-F 0 "#PWR02" H 4550 500 50  0001 C CNN
+F 0 "#PWR4" H 4550 500 50  0001 C CNN
 F 1 "+5V" H 4550 790 50  0000 C CNN
 F 2 "" H 4550 650 50  0001 C CNN
@@
 	4550 650  4550 1000
 $Comp
-L GND #PWR03
+L GND #PWR10
 U 1 1 5B7A7EFE
 P 8150 800
-F 0 "#PWR03" H 8150 550 50  0001 C CNN
+F 0 "#PWR10" H 8150 550 50  0001 C CNN
 F 1 "GND" H 8150 650 50  0000 C CNN
 F 2 "" H 8150 800 50  0001 C CNN
@@
 	8600 4950 8850 4950
 $Comp
-L GND #PWR04
+L GND #PWR11
 U 1 1 5B7C1985
 P 8600 5050
-F 0 "#PWR04" H 8600 4800 50  0001 C CNN
+F 0 "#PWR11" H 8600 4800 50  0001 C CNN
 F 1 "GND" H 8600 4900 50  0000 C CNN
 F 2 "" H 8600 5050 50  0001 C CNN
@@
 Connection ~ 4550 650
 $Comp
-L GND #PWR05
+L GND #PWR3
 U 1 1 5B7E4EA7
 P 3150 4300
-F 0 "#PWR05" H 3150 4050 50  0001 C CNN
+F 0 "#PWR3" H 3150 4050 50  0001 C CNN
 F 1 "GND" H 3150 4150 50  0000 C CNN
 F 2 "" H 3150 4300 50  0001 C CNN
@@
 	1750 1650 1750 2450
 $Comp
-L GND #PWR06
+L GND #PWR2
 U 1 1 5B7E721D
 P 1750 2450
-F 0 "#PWR06" H 1750 2200 50  0001 C CNN
+F 0 "#PWR2" H 1750 2200 50  0001 C CNN
 F 1 "GND" H 1750 2300 50  0000 C CNN
 F 2 "" H 1750 2450 50  0001 C CNN
@@
 $EndComp
 $Comp
-L GND #PWR07
+L GND #PWR5
 U 1 1 5B84307B
 P 5750 3550
-F 0 "#PWR07" H 5750 3300 50  0001 C CNN
+F 0 "#PWR5" H 5750 3300 50  0001 C CNN
 F 1 "GND" H 5750 3400 50  0000 C CNN
 F 2 "" H 5750 3550 50  0001 C CNN
@@
 	6750 3500 6950 3500
 $Comp
-L +5V #PWR08
+L +5V #PWR7
 U 1 1 5B84FD26
 P 6200 3050
-F 0 "#PWR08" H 6200 2900 50  0001 C CNN
+F 0 "#PWR7" H 6200 2900 50  0001 C CNN
 F 1 "+5V" H 6200 3190 50  0000 C CNN
 F 2 "" H 6200 3050 50  0001 C CNN
@@
 	1300 2400 1750 2400
 Connection ~ 1750 2400
-$Comp
-L Conn_01x02 J10
-U 1 1 5BFE94F1
-P 8900 2800
-F 0 "J10" H 8900 2900 50  0000 C CNN
-F 1 "m1-sensor" H 8900 2600 50  0000 C CNN
-F 2 "Connectors_Terminal_Blocks:TerminalBlock_Philmore_TB132_02x5mm_Straight" H 8900 2800 50  0001 C CNN
-F 3 "" H 8900 2800 50  0001 C CNN
-	1    8900 2800
-	-1   0    0    1
-$EndComp
-$Comp
-L Conn_01x02 J9
-U 1 1 5BFE95A9
-P 8900 2500
-F 0 "J9" H 8900 2600 50  0000 C CNN
-F 1 "m2-sensor" H 8900 2300 50  0000 C CNN
-F 2 "Connectors_Terminal_Blocks:TerminalBlock_Philmore_TB132_02x5mm_Straight" H 8900 2500 50  0001 C CNN
-F 3 "" H 8900 2500 50  0001 C CNN
-	1    8900 2500
-	-1   0    0    1
-$EndComp
-$Sheet
-S 9850 2250 1200 1400
-U 5BFF3A10
-F0 "Postion_control" 60
-F1 "file5BFF3A0F.sch" 60
-F2 "Left_pos_sens_1" I L 9850 2400 60
-F3 "Left_pos_sens_2" I L 9850 2700 60
-F4 "Right_pos_sens_2" I L 9850 2850 60
-F5 "Right_pos_sens_1" I L 9850 2550 60
-F6 "Left_pos_read_1" I L 9850 3050 60
-F7 "Left_pos_read_2" I L 9850 3350 60
-F8 "Right_pos_read_2" I L 9850 3500 60
-F9 "Right_pos_read_1" I L 9850 3200 60
-$EndSheet
-Wire Wire Line
-	9100 2400 9850 2400
-Wire Wire Line
-	9100 2500 9700 2500
-Wire Wire Line
-	9700 2500 9700 2550
-Wire Wire Line
-	9700 2550 9850 2550
-Wire Wire Line
-	9100 2700 9850 2700
-Wire Wire Line
-	9100 2800 9500 2800
 Wire Wire Line
 	9500 2800 9500 2850
 Wire Wire Line
-	9500 2850 9850 2850
+	9500 2850 10050 2850
 Wire Bus Line
 	9000 3950 8900 3950
@@
 	9450 3200 9850 3200
 Wire Wire Line
-	9450 3350 9850 3350
-Wire Wire Line
-	9450 3500 9850 3500
+	9450 3350 10050 3350
+Wire Wire Line
+	9450 3500 10050 3500
 Text Label 9550 3050 0    60   ~ 0
 SS
@@
 	8900 4600 8550 4600
 $Comp
-L +5V #PWR09
+L +5V #PWR9
 U 1 1 5C00CCE2
 P 8050 4650
-F 0 "#PWR09" H 8050 4500 50  0001 C CNN
+F 0 "#PWR9" H 8050 4500 50  0001 C CNN
 F 1 "+5V" H 8050 4790 50  0000 C CNN
 F 2 "" H 8050 4650 50  0001 C CNN
@@
 	1650 650  5200 650
 $Comp
-L +5V #PWR010
+L +5V #PWR6
 U 1 1 5C01C902
 P 5750 4550
-F 0 "#PWR010" H 5750 4400 50  0001 C CNN
+F 0 "#PWR6" H 5750 4400 50  0001 C CNN
 F 1 "+5V" H 5750 4690 50  0000 C CNN
 F 2 "" H 5750 4550 50  0001 C CNN
@@
 SCL
 $Comp
-L +5V #PWR?
+L +5V #PWR1
 U 1 1 5C06FAFE
 P 1550 4250
-F 0 "#PWR?" H 1550 4100 50  0001 C CNN
+F 0 "#PWR1" H 1550 4100 50  0001 C CNN
 F 1 "+5V" H 1550 4390 50  0000 C CNN
 F 2 "" H 1550 4250 50  0001 C CNN
@@
 $EndComp
 $Comp
-L R R?
+L R R2
 U 1 1 5C06FB93
 P 1800 4250
-F 0 "R?" V 1880 4250 50  0000 C CNN
+F 0 "R2" V 1880 4250 50  0000 C CNN
 F 1 "10k" V 1800 4250 50  0000 C CNN
 F 2 "Resistors_SMD:R_1206_HandSoldering" V 1730 4250 50  0001 C CNN
@@
 $EndComp
 $Comp
-L R R?
+L R R3
 U 1 1 5C06FDBF
 P 1800 4500
-F 0 "R?" V 1880 4500 50  0000 C CNN
+F 0 "R3" V 1880 4500 50  0000 C CNN
 F 1 "10k" V 1800 4500 50  0000 C CNN
 F 2 "Resistors_SMD:R_1206_HandSoldering" V 1730 4500 50  0001 C CNN
@@
 Text Label 2900 5700 0    60   ~ 0
 pwr_c1
+$Sheet
+S 10050 2300 900  1350
+U 5C1B51FD
+F0 "MotorsShield" 60
+F1 "Motors.sch" 60
+F2 "GND" I R 10950 3550 60
+F3 "d1sensor" I L 10050 3500 60
+F4 "m1black" I L 10050 2550 60
+F5 "m1sensor" I L 10050 2400 60
+F6 "d2sensor" I L 10050 3350 60
+F7 "m2black" I L 10050 2850 60
+F8 "m2sensor" I L 10050 2700 60
+F9 "vcc-in" I R 10950 3400 60
+$EndSheet
+$Comp
+L +5V #PWR12
+U 1 1 5C1BAB66
+P 11100 3300
+F 0 "#PWR12" H 11100 3150 50  0001 C CNN
+F 1 "+5V" H 11100 3440 50  0000 C CNN
+F 2 "" H 11100 3300 50  0001 C CNN
+F 3 "" H 11100 3300 50  0001 C CNN
+	1    11100 3300
+	1    0    0    -1
+$EndComp
+$Comp
+L GND #PWR13
+U 1 1 5C1BD542
+P 11100 3600
+F 0 "#PWR13" H 11100 3350 50  0001 C CNN
+F 1 "GND" H 11100 3450 50  0000 C CNN
+F 2 "" H 11100 3600 50  0001 C CNN
+F 3 "" H 11100 3600 50  0001 C CNN
+	1    11100 3600
+	1    0    0    -1
+$EndComp
+Wire Wire Line
+	10950 3400 11100 3400
+Wire Wire Line
+	11100 3400 11100 3300
+Wire Wire Line
+	11100 3600 11100 3550
+Wire Wire Line
+	11100 3550 10950 3550
+Connection ~ 8300 1400
+Connection ~ 8250 2150
+Wire Wire Line
+	9250 2800 9250 3050
+Wire Wire Line
+	9250 3050 8250 3050
+Wire Wire Line
+	8250 3050 8250 2150
+Connection ~ 9250 2800
+$Comp
+L Conn_01x03 J3
+U 1 1 5C1C6C52
+P 8800 1400
+F 0 "J3" H 8800 1600 50  0000 C CNN
+F 1 "m1" H 8800 1200 50  0000 C CNN
+F 2 "Connectors_Terminal_Blocks:TerminalBlock_Philmore_TB133_03x5mm_Straight" H 8800 1400 50  0001 C CNN
+F 3 "" H 8800 1400 50  0001 C CNN
+	1    8800 1400
+	1    0    0    -1
+$EndComp
+$Comp
+L Conn_01x03 J4
+U 1 1 5C1C7E9F
+P 8800 2100
+F 0 "J4" H 8800 2300 50  0000 C CNN
+F 1 "m2" H 8800 1900 50  0000 C CNN
+F 2 "Connectors_Terminal_Blocks:TerminalBlock_Philmore_TB133_03x5mm_Straight" H 8800 2100 50  0001 C CNN
+F 3 "" H 8800 2100 50  0001 C CNN
+	1    8800 2100
+	1    0    0    -1
+$EndComp
+Wire Wire Line
+	8600 1500 8600 1650
+Wire Wire Line
+	8600 1650 9900 1650
+Wire Wire Line
+	9900 1650 9900 2400
+Wire Wire Line
+	9900 2400 10050 2400
+Wire Wire Line
+	10050 2550 9800 2550
+Wire Wire Line
+	9800 2550 9800 1700
+Wire Wire Line
+	9800 1700 8300 1700
+Wire Wire Line
+	8300 1700 8300 1400
+Wire Wire Line
+	8450 2150 8450 2100
+Wire Wire Line
+	8450 2100 8600 2100
+Wire Wire Line
+	8600 2200 8600 2700
+Wire Wire Line
+	8600 2700 10050 2700
+Wire Wire Line
+	9500 2800 9250 2800
 $EndSCHEMATC

Commit message: prod
Connections:
- net labels added: RX, TX
- wire segments 145 -> 147
Changed lines of the file:
@@
 Wire Wire Line
 	9500 2800 9250 2800
+Wire Wire Line
+	4150 2650 4600 2650
+Wire Wire Line
+	4150 2750 4600 2750
+Text Label 4250 2650 0    60   ~ 0
+RX
+Text Label 4250 2750 0    60   ~ 0
+TX
 $EndSCHEMATC
